File: Hardware/SparkFun_RTK_mosaic-T.kicad_pcb (KiCad board)
At the start: 4 copper layers, 151.9 x 101.6 mm, 146 parts, among them J1 U.FL, J2 USB_C_Receptacle, J3 Qwiic_RA, J4 USB_C_Receptacle, J5 MagJack_PoE, J6 microSD, Q1 MBT3904DW1, Q3 BSS138, U1 ESP32-WROVER-IE-N16R8, U11 AP2112K-3.3, U2 mosaic-X5, U3 CH340C, U4 KSZ8041NL/I, U5 AP2112K-3.3

Commit message: More WIP
Parts:
- removed J3: Qwiic_RA, SparkFun-Connector:JST_SMD_1.0mm-4_RA
- removed TP_3V3P1, TP_5V1, TP_GND1: PTH, SparkFun-Connector:1x01
- added C32: 100uF, SparkFun-Capacitor:PANASONIC_D, F.Cu at (409.2, 79.8)
- added C33: 10uF, SparkFun-Capacitor:C_0603_1608Metric, F.Cu at (409.0, 103.8)
- added C34: 10uF, SparkFun-Capacitor:C_0603_1608Metric, F.Cu at (409.0, 106.3)
- added C35: 47uF, SparkFun-Capacitor:PANASONIC_D, F.Cu at (409.2, 87.5)
- added C36: 100uF, SparkFun-Capacitor:PANASONIC_D, F.Cu at (409.2, 95.2)
- added C37: 10uF, SparkFun-Capacitor:C_0603_1608Metric, F.Cu at (409.0, 108.8)
- added C38: 10uF, SparkFun-Capacitor:C_0603_1608Metric, F.Cu at (409.0, 111.3)
- added D10: BAT60A, SparkFun-Semiconductor-Standard:SOD-323, F.Cu at (413.4, 106.5)
- added D8: SK34A, SparkFun-Semiconductor-Standard:SMA, F.Cu at (410.6, 114.7)
- added D9: BAT60A, SparkFun-Semiconductor-Standard:SOD-323, F.Cu at (413.4, 103.8)
- added J7: Qwiic_Vertical, SparkFun-Connector:JST_SMD_1.0mm-4_Vertical, F.Cu at (421.6, 78.5)
- added JP_POE+_1: Measure, SparkFun-Jumper:Jumper_2_PTH_SMD_Combo-NC, F.Cu at (404.0, 103.7)
- added JP_POE-_1: Measure, SparkFun-Jumper:Jumper_2_PTH_SMD_Combo-NC, F.Cu at (404.0, 106.6)
- added JP_POE_1: ~, SparkFun-Jumper:Jumper_2_NC_Trace, F.Cu at (417.3, 101.6)
- added JP_VIN+_1: Measure, SparkFun-Jumper:Jumper_2_PTH_SMD_Combo-NC, F.Cu at (403.9, 110.0)
- added JP_VIN-_1: Measure, SparkFun-Jumper:Jumper_2_PTH_SMD_Combo-NC, F.Cu at (403.9, 113.0)
- added L3: 4.7uH, SparkFun-Coil:1008_2520Metric, F.Cu at (403.9, 116.2)
- added L4: 4.7uH, SparkFun-Coil:1008_2520Metric, F.Cu at (403.9, 119.6)
- added R36: 49.9, SparkFun-Resistor:R_1206_3216Metric, F.Cu at (409.8, 118.4)
- added TP_3V3P_1: PTH, SparkFun-Connector:1x01, F.Cu at (417.6, 104.8)
- added TP_5V_1: PTH, SparkFun-Connector:1x01, F.Cu at (417.6, 107.4)
- added TP_GND_1: PTH, SparkFun-Connector:1x01, F.Cu at (417.6, 110.0)
- added TP_VDC_1: PTH, SparkFun-Connector:1x01, F.Cu at (417.6, 112.6)
- added TP_VPOE_1: PTH, SparkFun-Connector:1x01, F.Cu at (417.6, 115.2)
- added U6: REC15E-2405SZ, SparkFun-Semiconductor-Standard:REC15E, F.Cu at (391.5, 89.2)
- added U7: Ag9905M, SparkFun-Semiconductor-Standard:Ag9900M, F.Cu at (390.3, 112.3)
- moved C27 1.43 mm to (311.1, 65.2)
- moved C7 1.20 mm to (312.4, 52.1)
- moved C22 1.15 mm to (308.6, 52.1)
- moved C29 1.12 mm to (316.2, 64.8)
- moved C3 1.12 mm to (326.4, 65.4)

Commit message: More WIP
Parts:
- removed ESP13/MTX1, ESP14/MRX1, ESP25/MRX4, ESP4/MTX4, MGPIO1, MGPIO2, MRX3, MTX3: 1.0mm, SparkFun-Connector:TestPoint-1.0mm
- removed JP_LINK1, JP_POE_1, JP_SHLD1, JP_SHLD2, JP_SPEED1: ~, SparkFun-Jumper:Jumper_2_NC_Trace
- removed JP_MEAS1, JP_POE+_1, JP_POE-_1, JP_VIN+_1, JP_VIN-_1: Measure, SparkFun-Jumper:Jumper_2_PTH_SMD_Combo-NC
- removed Q3: BSS138, SparkFun-Semiconductor-Standard:SOT23-3
- removed TP_1V8, TP_3V3, TP_3V3P_1, TP_5V_1, TP_GND_1, TP_VDC_1, TP_VDDA1, TP_VPOE_1: PTH, SparkFun-Connector:1x01
- added C39: 2.2uF, SparkFun-Capacitor:C_0603_1608Metric, F.Cu at (374.6, 158.4)
- added C40: 0.1uF, SparkFun-Capacitor:C_0603_1608Metric, F.Cu at (374.6, 160.9)
- added C41: 2.2uF, SparkFun-Capacitor:C_0603_1608Metric, F.Cu at (374.6, 163.4)
- added C42: 0.1uF, SparkFun-Capacitor:C_0603_1608Metric, F.Cu at (374.6, 165.9)
- added C43: 2.2uF, SparkFun-Capacitor:C_0603_1608Metric, F.Cu at (374.6, 168.4)
- added C44: 0.1uF, SparkFun-Capacitor:C_0603_1608Metric, F.Cu at (378.6, 158.4)
- added C45: 2.2uF, SparkFun-Capacitor:C_0603_1608Metric, F.Cu at (378.6, 160.9)
- added C46: 0.1uF, SparkFun-Capacitor:C_0603_1608Metric, F.Cu at (378.6, 163.4)
- added D11: CBI_LED_3mm_YGR, SparkFun-LED:CBI_LED_Triple_3mm_PTH, F.Cu at (370.8, 186.5)
- added D12: CBI_LED_3mm_YGR, SparkFun-LED:CBI_LED_Triple_3mm_PTH, F.Cu at (376.3, 186.5)
- added D13: DF5A5.6LFU, SparkFun-Semiconductor-Standard:SOT-353, F.Cu at (382.4, 167.8)
- added D14: DF5A5.6LFU, SparkFun-Semiconductor-Standard:SOT-353, F.Cu at (385.9, 167.8)
- added D15: PESD0402, SparkFun-Capacitor:C_0402_1005Metric, F.Cu at (380.5, 190.5)
- added J3: Val**, SparkFun-Connector:U.FL, F.Cu at (403.6, 156.2)
- added J8: Val**, SparkFun-Connector:RP-SMA_Edge, F.Cu at (391.2, 47.6)
- added J9: Screw_Cage_3.5mm-10, SparkFun-Connector:Screw_Cage_3.5mm-10, F.Cu at (152.9, 44.2)
- added JP10: ~, SparkFun-Jumper:Jumper_2_NC_Trace, B.Cu at (398.3, 60.3)
- added JP11: ~, SparkFun-Jumper:Jumper_2_NC_Trace, B.Cu at (398.3, 63.5)
- added JP12: ~, SparkFun-Jumper:Jumper_2_NC_Trace, B.Cu at (377.5, 54.9)
- added JP13: ~, SparkFun-Jumper:Jumper_2_NC_Trace, B.Cu at (377.5, 58.1)
- added JP2: Measure, SparkFun-Jumper:Jumper_2_PTH_SMD_Combo-NC, F.Cu at (378.4, 37.9)
- added JP3: Measure, SparkFun-Jumper:Jumper_2_PTH_SMD_Combo-NC, F.Cu at (378.4, 40.9)
- added JP4: Measure, SparkFun-Jumper:Jumper_2_PTH_SMD_Combo-NC, F.Cu at (378.4, 43.9)
- added JP5: Measure, SparkFun-Jumper:Jumper_2_PTH_SMD_Combo-NC, F.Cu at (378.4, 46.9)
- added JP6: Measure, SparkFun-Jumper:Jumper_2_PTH_SMD_Combo-NC, F.Cu at (378.4, 49.9)
- added JP7: ~, SparkFun-Jumper:Jumper_2_NC_Trace, B.Cu at (382.9, 48.4)
- added JP8: ~, SparkFun-Jumper:Jumper_2_NC_Trace, B.Cu at (398.3, 53.9)
- added JP9: ~, SparkFun-Jumper:Jumper_2_NC_Trace, B.Cu at (398.3, 57.1)
- added R37: 1k, SparkFun-Resistor:R_0603_1608Metric, F.Cu at (388.5, 146.2)
- added R38: 470, SparkFun-Resistor:R_0603_1608Metric, F.Cu at (381.1, 180.7)
- added R39: 470, SparkFun-Resistor:R_0603_1608Metric, F.Cu at (381.1, 183.2)
- added R40: 470, SparkFun-Resistor:R_0603_1608Metric, F.Cu at (381.1, 185.8)
- added R42: 470, SparkFun-Resistor:R_0603_1608Metric, F.Cu at (381.1, 188.3)
- added R43: 100k, SparkFun-Resistor:R_0603_1608Metric, F.Cu at (378.6, 165.9)
- added R44: 100k, SparkFun-Resistor:R_0603_1608Metric, F.Cu at (378.6, 168.4)
- added SW1: PTH_RA_h7.5mm, SparkFun-Switch:Push_PTH_RA_8-020_h7.5mm, F.Cu at (385.5, 138.0)
- added SW2: PTH_RA_h7.5mm, SparkFun-Switch:Push_PTH_RA_8-020_h7.5mm, F.Cu at (396.0, 138.0)
- added SW3: PTH_RA_h7.5mm, SparkFun-Switch:Push_PTH_RA_8-020_h7.5mm, F.Cu at (406.4, 138.0)
- added SW4: SPDT_Slide_SMD_7.2x3.5mm, SparkFun-Switch:Slide_DPDT_SMD_7.2x3.5mm, F.Cu at (384.7, 161.5)
- added TP1: PTH, SparkFun-Connector:1x01, F.Cu at (397.0, 37.7)
- added TP10: PTH, SparkFun-Connector:1x01, F.Cu at (388.0, 53.7)
- added TP11: PTH, SparkFun-Connector:1x01, F.Cu at (388.0, 56.3)
- added TP12: PTH, SparkFun-Connector:1x01, F.Cu at (388.0, 58.9)
- added TP13: PTH, SparkFun-Connector:1x01, F.Cu at (388.0, 61.5)
- added TP14: PTH, SparkFun-Connector:1x01, F.Cu at (388.0, 64.1)
- added TP15: PTH, SparkFun-Connector:1x01, F.Cu at (390.6, 53.7)
- added TP16: PTH, SparkFun-Connector:1x01, F.Cu at (390.6, 56.3)
- added TP17: PTH, SparkFun-Connector:1x01, F.Cu at (390.6, 58.9)
- added TP18: PTH, SparkFun-Connector:1x01, F.Cu at (390.6, 61.5)
- added TP19: PTH, SparkFun-Connector:1x01, F.Cu at (390.6, 64.1)
- added TP2: PTH, SparkFun-Connector:1x01, F.Cu at (382.4, 37.7)
- added TP20: PTH, SparkFun-Connector:1x01, F.Cu at (393.2, 53.7)
- added TP21: PTH, SparkFun-Connector:1x01, F.Cu at (393.2, 56.3)
- added TP22: PTH, SparkFun-Connector:1x01, F.Cu at (393.2, 58.9)
- added TP23: PTH, SparkFun-Connector:1x01, F.Cu at (380.6, 54.6)
- added TP3: PTH, SparkFun-Connector:1x01, F.Cu at (382.4, 40.3)
- added TP4: PTH, SparkFun-Connector:1x01, F.Cu at (382.4, 42.9)
- added TP7: PTH, SparkFun-Connector:1x01, F.Cu at (382.4, 45.5)
- added TP8: PTH, SparkFun-Connector:1x01, F.Cu at (401.4, 53.7)
- added TP9: PTH, SparkFun-Connector:1x01, F.Cu at (401.4, 56.3)
- added U10: 74LVC2T45DC, SparkFun-Semiconductor-Standard:VSSOP8_SOT765-1, F.Cu at (370.3, 166.9)
- added U12: 74LVC2T45DC, SparkFun-Semiconductor-Standard:VSSOP8_SOT765-1, F.Cu at (370.3, 170.7)
- added U8: 74LVC2T45DC, SparkFun-Semiconductor-Standard:VSSOP8_SOT765-1, F.Cu at (370.3, 159.3)
- added U9: 74LVC2T45DC, SparkFun-Semiconductor-Standard:VSSOP8_SOT765-1, F.Cu at (370.3, 163.1)
- C1, C2, C21, C22, C23, C27, C28, C29, C3, C4, C5, C7, C8, L1, Q1, R1, R11, R2, R3, R4, R6, R7, R8, U11, U3, U5: moved to F.Cu
- D1: value TVS_0402 -> PESD0402
- FID1, FID2, FID3, FID4: value Fiducial_0.5 -> Fiducial_0.5mm
- J1: value U.FL -> Val**; footprint SparkFun-Connector:U.FL -> SparkFun-Connector:SMA_Edge
- R12, R13: value 2.2k -> 470; footprint SparkFun-Resistor:R_0402_1005Metric -> SparkFun-Resistor:R_0603_1608Metric; moved to F.Cu
- R16, R41: value 169k -> 100k; moved to F.Cu
- R5: footprint SparkFun-Resistor:R_0402_1005Metric -> SparkFun-Resistor:R_0603_1608Metric; moved to F.Cu
- ST1, ST2, ST3, ST4: value Standoff -> STAND-OFF
- TR1: value RFCMF1220100M4T -> Val**; moved to F.Cu
- moved R13 151.8 mm to (381.1, 178.2), turned to 0 degrees
- moved R12 145.1 mm to (381.1, 175.7), turned to 0 degrees
- moved J1 9.12 mm to (297.2, 36.8), turned to 0 degrees
- moved R11 7.31 mm to (330.0, 65.4), turned to 180 degrees
- moved R41 6.10 mm to (329.2, 41.5)
- moved C2 5.59 mm to (296.8, 58.5)
- moved C8 5.59 mm to (296.8, 54.6)
- moved R1 5.59 mm to (296.8, 56.6)
- moved R2 5.59 mm to (301.9, 46.9), turned to 0 degrees
- moved R3 5.59 mm to (301.9, 47.9), turned to 0 degrees
- moved C27 5.08 mm to (316.2, 65.2)
- moved C29 5.08 mm to (311.1, 64.8)
- moved C22 3.81 mm to (312.4, 52.1)
- moved C7 3.81 mm to (308.6, 52.1)
- moved C21 3.56 mm to (308.5, 59.6), turned to 180 degrees
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Connections:
- C8 pad 1: ESP~{RST} -> ESP_~{RST}
- Q1 pad 3: ESP~{RST} -> ESP_~{RST}
- R1 pad 2: ESP~{RST} -> ESP_~{RST}
- R12 pad 1: 1.8V -> Net-(D11-PadANODE_1)
- R12 pad 2: MPPS -> ESP32/LED_ERROR
- R13 pad 1: 3.3V_P -> Net-(D11-PadANODE_2)
- R13 pad 2: MPPS_3V3 -> ESP33/LED_LOCK
- R16 pad 1: MEventA -> VCCIO
- R16 pad 2: Net-(U2-EVENTA) -> MCTS2_I
- R41 pad 1: MEventB -> VCCIO
- R41 pad 2: Net-(U2-EVENTB) -> MRX2_I
- TP5 pad 1: ESP~{RST} -> 3.3V
- TP6 pad 1: MPPS_3V3 -> GND
- U1 pad 11: unconnected-(U1-IOA26-Pad11) -> ESP26/MCTS1
- U1 pad 12: unconnected-(U1-IOA27-Pad12) -> ESP27/MRTS1
- U1 pad 3: ESP~{RST} -> ESP_~{RST}
- U1 pad 8: unconnected-(U1-IOA32-Pad8) -> ESP32/LED_ERROR
- U1 pad 9: unconnected-(U1-IOA33-Pad9) -> ESP33/LED_LOCK
- U2 pad AC6: Net-(U2-EVENTA) -> MEventA_1V8
- U2 pad AC7: Net-(U2-EVENTB) -> MEventB_1V8
- U2 pad AC8: MPPS -> MPPS_1V8
- U2 pad C1: unconnected-(U2-COM1_RTS-PadC1) -> ESP27/MRTS1
- U2 pad E1: unconnected-(U2-COM1_CTS-PadE1) -> ESP26/MCTS1
- U2 pad L1: unconnected-(U2-COM3_RTS-PadL1) -> Net-(U2-COM3_RTS)
- U2 pad N1: unconnected-(U2-COM3_CTS-PadN1) -> Net-(U2-COM3_CTS)

Commit message: More WIP
Parts:
- added C47: 0.1uF, SparkFun-Capacitor:C_0603_1608Metric, F.Cu at (423.8, 125.8)
- added C48: 10uF, SparkFun-Capacitor:C_0603_1608Metric, F.Cu at (423.8, 128.3)
- added U13: SiT5358AI-FS033IT-10.000000, SparkFun-Semiconductor-Standard:Ceramic_QFN_5.0x3.2mm-10, F.Cu at (426.0, 122.0)
- J1: value Val** -> SMA_Edge
- J3: value Val** -> U.FL
- J8: value Val** -> RP-SMA_Edge
- ST1, ST2, ST3, ST4: value STAND-OFF -> Standoff
- TR1: value Val** -> RFCMF1220100M4T

Commit message: PCB WIP
Parts:
- added C49: 2.2uF, SparkFun-Capacitor:C_0603_1608Metric, F.Cu at (319.2, 172.1)
- added C50: 0.1uF, SparkFun-Capacitor:C_0603_1608Metric, F.Cu at (319.2, 174.7)
- added C51: 2.2uF, SparkFun-Capacitor:C_0603_1608Metric, F.Cu at (319.2, 177.2)
- added C52: 0.1uF, SparkFun-Capacitor:C_0603_1608Metric, F.Cu at (319.2, 179.7)
- added C53: 10uF, SparkFun-Capacitor:C_0402_1005Metric, F.Cu at (346.7, 179.6)
- added C54: 0.1uF, SparkFun-Capacitor:C_0603_1608Metric, F.Cu at (343.9, 177.3)
- added C55: 1.0nF, SparkFun-Capacitor:C_0603_1608Metric, F.Cu at (319.2, 182.2)
- added C56: 1.0nF, SparkFun-Capacitor:C_0603_1608Metric, F.Cu at (319.2, 184.7)
- added C57: 1.0nF, SparkFun-Capacitor:C_0603_1608Metric, F.Cu at (323.2, 172.1)
- added C58: 1.0nF, SparkFun-Capacitor:C_0603_1608Metric, F.Cu at (323.2, 174.7)
- added C59: 27pF, SparkFun-Capacitor:C_0603_1608Metric, F.Cu at (323.2, 177.2)
- added J11: SMA_Edge, SparkFun-Connector:SMA_Edge, F.Cu at (321.7, 196.4)
- added J12: SMA_Edge, SparkFun-Connector:SMA_Edge, F.Cu at (330.8, 196.4)
- added JP14: ~, SparkFun-Jumper:Jumper_3_NC-2_Trace, F.Cu at (345.8, 193.6)
- added JP15: ~, SparkFun-Jumper:Jumper_2_NO, F.Cu at (343.6, 180.2)
- added JP16: ~, SparkFun-Jumper:Jumper_2_NC_Trace, B.Cu at (111.0, 142.2)
- added JP17: ~, SparkFun-Jumper:Jumper_2_NC_Trace, B.Cu at (111.0, 144.8)
- added JP18: ~, SparkFun-Jumper:Jumper_2_NC_Trace, B.Cu at (111.0, 147.3)
- added JP19: ~, SparkFun-Jumper:Jumper_2_NC_Trace, B.Cu at (125.2, 142.2)
- added JP20: ~, SparkFun-Jumper:Jumper_2_NC_Trace, B.Cu at (125.2, 144.8)
- added JP21: ~, SparkFun-Jumper:Jumper_2_NC_Trace, B.Cu at (125.2, 147.3)
- added L5: 10uH, SparkFun-Capacitor:C_0805_2012Metric, F.Cu at (331.4, 183.9)
- added L6: 130nH, SparkFun-Capacitor:C_0603_1608Metric, F.Cu at (323.2, 179.7)
- added L7: 130nH, SparkFun-Capacitor:C_0603_1608Metric, F.Cu at (323.2, 182.2)
- added R45: 49.9, SparkFun-Resistor:R_0603_1608Metric, F.Cu at (323.2, 184.7)
- added R46: 2.2k, SparkFun-Resistor:R_0402_1005Metric, F.Cu at (344.9, 198.7)
- added R47: 2.2k, SparkFun-Resistor:R_0402_1005Metric, F.Cu at (344.9, 200.7)
- added R48: 49.9, SparkFun-Resistor:R_0603_1608Metric, F.Cu at (327.2, 172.1)
- added R49: 49.9, SparkFun-Resistor:R_0603_1608Metric, F.Cu at (327.2, 174.7)
- added R50: 49.9, SparkFun-Resistor:R_0603_1608Metric, F.Cu at (327.2, 177.2)
- added R51: 0, SparkFun-Resistor:R_0603_1608Metric, F.Cu at (345.5, 196.4)
- added TP24: PTH, SparkFun-Connector:1x01, F.Cu at (343.2, 172.2)
- added TP25: PTH, SparkFun-Connector:1x01, F.Cu at (343.2, 174.8)
- added TP26: PTH, SparkFun-Connector:1x01, F.Cu at (345.8, 172.2)
- added TP27: PTH, SparkFun-Connector:1x01, F.Cu at (339.6, 193.3)
- added TP28: PTH, SparkFun-Connector:1x01, F.Cu at (339.6, 195.9)
- added TP29: PTH, SparkFun-Connector:1x01, F.Cu at (339.6, 198.5)
- added TP30: PTH, SparkFun-Connector:1x01, F.Cu at (339.6, 201.1)
- added TP31: PTH, SparkFun-Connector:1x01, F.Cu at (342.2, 193.3)
- added TP32: PTH, SparkFun-Connector:1x01, F.Cu at (342.2, 195.9)
- added TP33: PTH, SparkFun-Connector:1x01, F.Cu at (342.2, 198.5)
- added TP34: PTH, SparkFun-Connector:1x01, F.Cu at (318.5, 202.4)
- added TP35: PTH, SparkFun-Connector:1x01, F.Cu at (318.5, 205.0)
- added TP36: PTH, SparkFun-Connector:1x01, F.Cu at (321.1, 202.4)
- added TP37: PTH, SparkFun-Connector:1x01, F.Cu at (321.1, 205.0)
- added TP38: PTH, SparkFun-Connector:1x01, F.Cu at (323.7, 202.4)
- added TP39: PTH, SparkFun-Connector:1x01, F.Cu at (323.7, 205.0)
- added TP40: PTH, SparkFun-Connector:1x01, F.Cu at (335.0, 183.7)
- added TP41: PTH, SparkFun-Connector:1x01, F.Cu at (345.8, 174.8)
- added TP42: PTH, SparkFun-Connector:1x01, F.Cu at (348.4, 172.2)
- added TP43: PTH, SparkFun-Connector:1x01, F.Cu at (348.4, 174.8)
- added U14: 74LVC2T45DC, SparkFun-Semiconductor-Standard:VSSOP8_SOT765-1, F.Cu at (331.5, 173.0)
- added U15: 74LVC2T45DC, SparkFun-Semiconductor-Standard:VSSOP8_SOT765-1, F.Cu at (331.5, 176.8)
- added U16: 74LVC2T45DC, SparkFun-Semiconductor-Standard:VSSOP8_SOT765-1, F.Cu at (331.5, 180.6)
- C47: value 0.1uF -> 10uF
- C48: value 10uF -> 0.1uF
- R30: value 1k -> 33
- R31: value 1k -> 0
- R32: value 33 -> 0
- R8: value 4.7k -> 1k
- moved R38 274.1 mm to (110.5, 137.2), turned to 90 degrees
- moved SW3 272.0 mm to (134.6, 149.5)
- moved R13 271.2 mm to (113.0, 137.2), turned to 90 degrees
- moved R12 268.3 mm to (115.6, 137.2), turned to 90 degrees
- moved R39 264.5 mm to (120.7, 137.2), turned to 90 degrees
- moved R40 262.4 mm to (123.2, 137.2), turned to 90 degrees
- moved R42 260.4 mm to (125.7, 137.2), turned to 90 degrees
- moved D12 257.9 mm to (120.7, 152.4)
- moved D11 257.5 mm to (115.6, 152.4)
- moved R37 254.4 mm to (134.2, 137.2), turned to -90 degrees
- moved J7 251.9 mm to (177.8, 142.2), turned to 180 degrees
- moved J6 203.4 mm to (148.6, 150.4)
- moved J5 202.8 mm to (116.8, 60.2), turned to 180 degrees
- moved SW1 167.4 mm to (218.4, 148.6)
- moved SW2 155.1 mm to (241.3, 149.5)
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Connections:
- net /50Ohm renamed Net-(D15-A2)
- C24 pad 1: 10MHz -> REF_IN
- D11 pad ANODE_1: Net-(D11-PadANODE_1) -> Net-(JP16-B)
- D11 pad ANODE_2: Net-(D11-PadANODE_2) -> Net-(JP17-B)
- D11 pad ANODE_3: Net-(D11-PadANODE_3) -> Net-(JP18-B)
- D12 pad ANODE_1: Net-(D12-PadANODE_1) -> Net-(JP19-B)
- D12 pad ANODE_2: Net-(D12-PadANODE_2) -> Net-(JP20-B)
- D12 pad ANODE_3: Net-(D12-PadANODE_3) -> Net-(JP21-B)
- D14 pad 5: VCCIO -> unconnected-(D14-K4-Pad5)
- J9 pad 4: MRX2_I -> MCTS2_I
- J9 pad 5: MTX2_O -> MRTS2_O
- J9 pad 6: MRTS2_O -> MTX2_O
- J9 pad 7: MCTS2_I -> MRX2_I
- R12 pad 1: Net-(D11-PadANODE_1) -> Net-(JP16-A)
- R13 pad 1: Net-(D11-PadANODE_2) -> Net-(JP17-A)
- R30 pad 1: 10MHz -> REF_IN
- R30 pad 2: 10MHz -> Net-(U14-1B)
- R31 pad 1: 10MHz -> Net-(C55-Pad1)
- R31 pad 2: GND -> Net-(R31-Pad2)
- R32 pad 1: 10MHz -> Net-(J11-In)
- R32 pad 2: 10MHz -> Net-(C57-Pad1)
- R34 pad 2: SPEED -> LINK
- R35 pad 2: LINK -> SPEED
- R38 pad 1: Net-(D11-PadANODE_3) -> Net-(JP18-A)
- R39 pad 1: Net-(D12-PadANODE_1) -> Net-(JP19-A)
- R40 pad 1: Net-(D12-PadANODE_2) -> Net-(JP20-A)
- R42 pad 1: Net-(D12-PadANODE_3) -> Net-(JP21-A)
- U1 pad 30: unconnected-(U1-IO18-Pad30) -> ESP18/SDA2
- U1 pad 31: unconnected-(U1-IO19-Pad31) -> ESP19/SCL2
- U1 pad 37: unconnected-(U1-IO23-Pad37) -> Net-(U1-IO23)
- U1 pad 5: unconnected-(U1-IA39-Pad5) -> Net-(U1-IA39)
- U1 pad 6: unconnected-(U1-IA34-Pad6) -> Net-(U1-IA34)
- U13 pad 10: ESP21/SDA -> ESP18/SDA2
- U13 pad 2: ESP22/SCL -> ESP19/SCL2
- U13 pad 6: unconnected-(U13-CLK-Pad6) -> Net-(U13-CLK)
- U2 pad AC17: 10MHz -> REF_IN
- U4 pad 30: SPEED -> LINK
- U4 pad 31: LINK -> SPEED
Other:
- board size 151.9 x 101.6 mm -> 151.8 x 101.6 mm

Commit message: Board edge components placed
Parts:
- moved J11 188.4 mm to (199.4, 53.1)
- moved J12 180.1 mm to (221.6, 53.1)
- moved J8 147.5 mm to (243.8, 53.1)
- moved J1 121.1 mm to (177.2, 53.1)
- moved FID2 3.59 mm to (106.7, 147.3)
- moved FID3 3.59 mm to (106.7, 147.3)
- moved FID1 3.59 mm to (248.9, 55.9)
- moved FID4 3.59 mm to (248.9, 55.9)
Other:
- board text added: "V-Score To V-Score"

Commit message: Ready for airwire review
Parts:
- removed R46, R47: 2.2k, SparkFun-Resistor:R_0402_1005Metric
- removed the kibuzzard-65A7F440 at (340.4, 66.0)
- removed kibuzzard-65A7F47C: G***, kibuzzard-65A7F47C
- removed kibuzzard-65A7F4E8: G***, kibuzzard-65A7F4E8
- removed kibuzzard-65A7F60E: G***, kibuzzard-65A7F60E
- removed kibuzzard-65A7F63F: G***, kibuzzard-65A7F63F
- removed kibuzzard-65A7F686: G***, kibuzzard-65A7F686
- removed kibuzzard-65A7F697: G***, kibuzzard-65A7F697
- added C60: 0.1uF, SparkFun-Capacitor:C_0603_1608Metric, F.Cu at (182.1, 137.2)
- added C62: 0.1uF, SparkFun-Capacitor:C_0603_1608Metric, F.Cu at (214.9, 60.7)
- added C63: 0.1uF, SparkFun-Capacitor:C_0603_1608Metric, F.Cu at (221.5, 57.7)
- added C64: 2.2uF, SparkFun-Capacitor:C_0603_1608Metric, F.Cu at (203.5, 62.2)
- added C65: 2.2uF, SparkFun-Capacitor:C_0603_1608Metric, F.Cu at (195.3, 62.2)
- added C66: 0.1uF, SparkFun-Capacitor:C_0603_1608Metric, F.Cu at (201.9, 62.2)
- added C67: 0.1uF, SparkFun-Capacitor:C_0603_1608Metric, F.Cu at (196.8, 62.2)
- added kibuzzard-65A7F891: G***, kibuzzard-65A7F891, B.Cu at (225.2, 69.8)
- C1, C2, C4, C5, C53, C8: footprint SparkFun-Capacitor:C_0402_1005Metric -> SparkFun-Capacitor:C_0603_1608Metric
- C54: value 0.1uF -> 2.2uF
- G*** (x2), JP7, Ref**: moved to F.Cu
- G***, JP14, JP15, JP2, JP3, JP4, JP5: moved to B.Cu
- R1, R2, R3, R4, R6, R7, R8: footprint SparkFun-Resistor:R_0402_1005Metric -> SparkFun-Resistor:R_0603_1608Metric
- R31, R32: value 0 -> 2.2k
- moved D8 300.2 mm to (110.5, 110.5)
- moved C35 300.2 mm to (110.5, 116.8), turned to -90 degrees
- moved C36 274.6 mm to (134.6, 95.1), turned to -90 degrees
- moved U7 270.7 mm to (120.7, 88.9), turned to 90 degrees
- moved JP5 270.5 mm to (109.2, 73.7), turned to -90 degrees
- moved C37 269.6 mm to (139.7, 96.5), turned to 90 degrees
- moved JP4 268.3 mm to (111.8, 73.7), turned to -90 degrees
- moved C38 267.0 mm to (142.2, 100.3), turned to 90 degrees
- moved C32 266.1 mm to (147.3, 127.0), turned to 180 degrees
- moved R36 265.9 mm to (144.8, 97.6), turned to 90 degrees
- moved JP13 265.7 mm to (111.8, 53.3), turned to 0 degrees
- moved D9 265.0 mm to (148.6, 114.3), turned to 180 degrees
- moved L4 264.9 mm to (139.7, 100.3), turned to -90 degrees
- moved D10 264.8 mm to (148.6, 106.7), turned to 180 degrees
- moved U6 264.7 mm to (128.3, 116.8)
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Connections:
- C54 pad 1: VCCIO -> 3.3V
- D13 pad 1: MCTS2_I -> MRTS2_O
- D13 pad 3: MRX2_I -> MTX2_O
- D13 pad 4: MTX2_O -> MRX2_I
- D13 pad 5: MRTS2_O -> MCTS2_I
- D14 pad 4: MPPS_O -> unconnected-(D14-K3-Pad4)
- D14 pad 5: unconnected-(D14-K4-Pad5) -> MPPS_O
- R31 pad 1: Net-(C55-Pad1) -> Net-(JP14-B)
- R31 pad 2: Net-(R31-Pad2) -> ESP18/SDA2
- R32 pad 1: Net-(J11-In) -> Net-(JP14-A)
- R32 pad 2: Net-(C57-Pad1) -> ESP19/SCL2
- R4 pad 1: Net-(JP1-B) -> ESP21/SDA
- R4 pad 2: ESP21/SDA -> Net-(JP1-B)
- R49 pad 1: Net-(R31-Pad2) -> Net-(C62-Pad1)
- R50 pad 1: Net-(R31-Pad2) -> Net-(C62-Pad1)
- R6 pad 1: Net-(JP1-A) -> ESP22/SCL
- R6 pad 2: ESP22/SCL -> Net-(JP1-A)
Routing:
- added copper zone on B.Cu, net GND-ISO
- added copper zone on F.Cu, net GND-ISO
- added copper zone on In1.Cu, net GND-ISO
- added copper zone on In2.Cu, net GND-ISO
Other:
- board text removed: "Route Out"
