File: Hardware/SparkFun_RTK_mosaic-T.kicad_pcb (KiCad board)
At the start: 4 copper layers, 151.8 x 101.6 mm, 328 parts, among them J1 SMA_Edge, J11 SMA_Edge, J12 SMA_Edge, J2 USB_C_Receptacle, J3 U.FL, J4 USB_C_Receptacle, J5 MagJack_PoE, J6 microSD, J7 Qwiic_Vertical, J8 RP-SMA_Edge, J9 Screw_Cage_3.5mm-10, Q1 MBT3904DW1, SW1 PTH_RA_h7.5mm, SW2 PTH_RA_h7.5mm, SW3 PTH_RA_h7.5mm, SW4 SPDT_Slide_SMD_7.2x3.5mm, U1 ESP32-WROVER-IE-N16R8, U10 74LVC2T45DC, U11 AP2112K-3.3, U12 74LVC2T45DC, U13 SiT5358AI-FS033IT-10.000000, U14 74LVC2T45DC, U15 74LVC2T45DC, U16 74LVC2T45DC, U2 mosaic-X5, U3 CH340C, U4 KSZ8041NL/I, U5 AP2112K-3.3, U6 REC15E-2405SZ, U7 Ag9905M, U8 74LVC2T45DC, U9 74LVC2T45DC

Commit message: Ready for routing
Parts:
- added kibuzzard-66A21191: G***, kibuzzard-66A21191, B.Cu at (114.8, 53.3)
- added kibuzzard-66A211A5: G***, kibuzzard-66A211A5, B.Cu at (125.7, 53.3)
- added kibuzzard-66A21255: G***, kibuzzard-66A21255, F.Cu at (142.2, 93.7)
- added kibuzzard-66A2129F: G***, kibuzzard-66A2129F, B.Cu at (143.3, 60.2)
- added kibuzzard-66A212C6: G***, kibuzzard-66A212C6, B.Cu at (153.7, 64.5)
- added kibuzzard-66A212DB: G***, kibuzzard-66A212DB, B.Cu at (146.8, 60.2)
- added kibuzzard-66A212E8: G***, kibuzzard-66A212E8, B.Cu at (150.4, 60.5)
- added kibuzzard-66A212F8: G***, kibuzzard-66A212F8, B.Cu at (140.0, 60.7)
- added kibuzzard-66A21305: G***, kibuzzard-66A21305, B.Cu at (157.2, 61.7)
- added kibuzzard-66A21310: G***, kibuzzard-66A21310, B.Cu at (160.8, 61.7)
- added kibuzzard-66A2131B: G***, kibuzzard-66A2131B, B.Cu at (164.3, 60.5)
- added kibuzzard-66A21341: G***, kibuzzard-66A21341, F.Cu at (204.7, 53.1)
- added kibuzzard-66A21351: G***, kibuzzard-66A21351, F.Cu at (215.6, 53.1)
- added kibuzzard-66A21378: G***, kibuzzard-66A21378, F.Cu at (239.0, 57.7)
- J1, J11, J12: value SMA_Edge -> Val**
- J3: value U.FL -> Val**
- J8: value RP-SMA_Edge -> Val**
- ST1, ST2, ST3, ST4: value Standoff -> STAND-OFF
- TR1: value RFCMF1220100M4T -> Val**
