File: Hardware/USB.kicad_sch (KiCad schematic)
At the start: 17 parts, among them J2 USB_C_Receptacle, J4 USB_C_Receptacle, Q1 MBT3904DW1, U3 CH340C

Commit message: More WIP
Parts:
- added JP10, JP11: ~, SparkFun-Jumper:Jumper_2_NC_Trace, symbol SparkFun-Jumper:SolderJumper_2_Bridged
- added R37: 1k, SparkFun-Resistor:R_0603_1608Metric, symbol SparkFun-Resistor:1k_0603
- added SW1, SW2, SW3: PTH_RA_h7.5mm, SparkFun-Switch:Push_PTH_RA_8-020_h7.5mm, symbol SparkFun-Switch:SPST_Push_PTH_RA_h7.5mm
- added TP8, TP9: PTH, SparkFun-Connector:1x01, symbol SparkFun-Connector:TestPoint_PTH
- renumbered JP_SHLD1 to JP8, JP_SHLD2 to JP9
Connections:
- net ESP0/BOOT: now also JP11.2 (B)
- net GND: now also SW1.1, SW2.1, SW3.1
- net VUSB: now also TP8.1
- net VUSB2: now also TP9.1
- net ESP~{RST} renamed ESP_~{RST}
- net ESP_~{RST}: now also JP10.2 (B)
- new net: JP10.1 (A), SW1.2
- new net: R37.2, SW3.2
- new net: JP11.1 (A), SW2.2
- new net LOG_BTN: R37.1
Other:
- note added: "Buttons"
- moved on the sheet: C4, C5, Q1A, Q1B, R2, R3, U3

Commit message: More WIP
Other:
- moved on the sheet: C4, C5, Q1A, Q1B, R2, R3, U3

Commit message: More WIP
Changed lines of the file:
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@@
 	(text "Buttons"
 		(exclude_from_sim no)
-		(at 214.63 113.03 0)
+		(at 214.63 111.76 0)
 		(effects
 			(font

Commit message: Schematic complete
Parts:
- added TP34, TP35, TP36, TP37, TP38, TP39: PTH, SparkFun-Connector:1x01, symbol SparkFun-Connector:TestPoint_PTH
Connections:
- net CH340-~{DTR}: now also TP38.1
- net CH340-~{RTS}: now also TP39.1
- net ESP0/BOOT: now also TP36.1
- net ESP1/CH340-RX: now also TP35.1
- net ESP3/CH340-TX: now also TP34.1
- net ESP_~{RST}: now also TP37.1

Commit message: Ready for airwire review
Parts:
- removed C4: 2.2uF, SparkFun-Capacitor:C_0402_1005Metric, symbol SparkFun-Capacitor:2.2uF_0402_10V_10%
- removed C5: 0.1uF, SparkFun-Capacitor:C_0402_1005Metric, symbol SparkFun-Capacitor:0.1uF_0402_6.3V_10%
- removed R2, R3: 10k, SparkFun-Resistor:R_0402_1005Metric, symbol SparkFun-Resistor:10k_0402
- added C4: 2.2uF, SparkFun-Capacitor:C_0603_1608Metric, symbol SparkFun-Capacitor:2.2uF_0603_10V_20%
- added C5: 0.1uF, SparkFun-Capacitor:C_0603_1608Metric, symbol SparkFun-Capacitor:0.1uF_0603_25V_20%
- added R2, R3: 10k, SparkFun-Resistor:R_0603_1608Metric, symbol SparkFun-Resistor:10k_0603
Connections:
- net 3.3V: now also C4.1, C5.1
- net CH340-~{DTR}: now also R2.2
- net CH340-~{RTS}: now also R3.2
- net GND: now also C4.2, C5.2
- net at Q1.2 (B1): now also R3.1
- net at Q1.5 (B2): now also R2.1

Commit message: Routing WIP
Connections:
- net ESP_DM: now also D3.3 (I/O2); no longer D3.1 (I/O1)
- net ESP_DP: now also D3.1 (I/O1); no longer D3.3 (I/O2)
- net MOSAIC_DM: now also TR1.2; no longer TR1.4
- net MOSAIC_DP: now also TR1.4; no longer TR1.2
- net at D2.3 (I/O2), TR1.1: now also J2.A7 (D-), J2.B7 (D-); no longer J2.A6 (D+), J2.B6 (D+)
- net at D2.1 (I/O1), TR1.3: now also J2.A6 (D+), J2.B6 (D+); no longer J2.A7 (D-), J2.B7 (D-)
Other:
- note added: "USB Track Impedance: Differential Pair https://saturnpcb.com/saturn-pcb-toolkit/ Prepreg thickness: 8.3 mil (JLC7628). Er = 4.6 10.5 mil track with 9.5 mil gap (20 mil center to center) = 90 Ohms"
Changed lines of the file:
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@@
-	)
-	(junction
-		(at 80.01 52.07)
-		(diameter 0)
-		(color 0 0 0 0)
 	)
 	(junction
@@
 	)
 	(junction
-		(at 91.44 132.08)
+		(at 207.01 55.88)
 		(diameter 0)
 		(color 0 0 0 0)
 	)
 	(junction
-		(at 201.93 55.88)
+		(at 80.01 54.61)
+		(diameter 0)
+		(color 0 0 0 0)
+	)
+	(junction
+		(at 91.44 132.08)
 		(diameter 0)
 		(color 0 0 0 0)
@@
 	)
 	(junction
+		(at 201.93 53.34)
+		(diameter 0)
+		(color 0 0 0 0)
+	)
+	(junction
 		(at 132.08 132.08)
 		(diameter 0)
@@
 	)
 	(junction
-		(at 207.01 53.34)
+		(at 74.93 52.07)
 		(diameter 0)
 		(color 0 0 0 0)
 	)
-	(junction
-		(at 74.93 54.61)
-		(diameter 0)
-		(color 0 0 0 0)
-	)
 	(wire
 		(pts
@@
 	(wire
 		(pts
-			(xy 195.58 53.34) (xy 207.01 53.34)
-		)
-		(stroke
-			(width 0)
-			(type default)
-		)
-	)
-	(wire
-		(pts
 			(xy 240.03 125.73) (xy 241.3 125.73)
 		)
@@
 	(polyline
 		(pts
-			(xy 12.7 99.06) (xy 266.7 99.06)
+			(xy 12.7 102.87) (xy 266.7 102.87)
 		)
 		(stroke
@@
 	(polyline
 		(pts
-			(xy 137.16 99.06) (xy 137.16 12.7)
+			(xy 137.16 102.87) (xy 137.16 12.7)
 		)
 		(stroke
@@
 	(wire
 		(pts
+			(xy 201.93 53.34) (xy 213.36 53.34)
+		)
+		(stroke
+			(width 0)
+			(type default)
+		)
+	)
+	(wire
+		(pts
 			(xy 195.58 64.77) (xy 198.12 64.77)
 		)
@@
 	(wire
 		(pts
+			(xy 201.93 34.29) (xy 201.93 53.34)
+		)
+		(stroke
+			(width 0)
+			(type default)
+		)
+	)
+	(wire
+		(pts
 			(xy 203.2 127) (xy 203.2 125.73)
 		)
@@
 	(wire
 		(pts
-			(xy 207.01 53.34) (xy 213.36 53.34)
+			(xy 195.58 53.34) (xy 201.93 53.34)
 		)
 		(stroke
@@
 	(wire
 		(pts
-			(xy 195.58 55.88) (xy 201.93 55.88)
+			(xy 195.58 55.88) (xy 207.01 55.88)
 		)
 		(stroke
@@
 	(wire
 		(pts
+			(xy 96.52 54.61) (xy 99.06 54.61)
+		)
+		(stroke
+			(width 0)
+			(type default)
+		)
+	)
+	(wire
+		(pts
 			(xy 208.28 34.29) (xy 201.93 34.29)
 		)
@@
 	(wire
 		(pts
-			(xy 68.58 54.61) (xy 74.93 54.61)
-		)
-		(stroke
-			(width 0)
-			(type default)
-		)
-	)
-	(wire
-		(pts
-			(xy 68.58 52.07) (xy 80.01 52.07)
+			(xy 68.58 54.61) (xy 80.01 54.61)
+		)
+		(stroke
+			(width 0)
+			(type default)
+		)
+	)
+	(wire
+		(pts
+			(xy 68.58 52.07) (xy 74.93 52.07)
 		)
 		(stroke
@@
 	(wire
 		(pts
+			(xy 80.01 54.61) (xy 86.36 54.61)
+		)
+		(stroke
+			(width 0)
+			(type default)
+		)
+	)
+	(wire
+		(pts
 			(xy 132.08 130.81) (xy 132.08 132.08)
 		)
@@
 	(wire
 		(pts
-			(xy 96.52 54.61) (xy 99.06 54.61)
+			(xy 80.01 45.72) (xy 80.01 54.61)
+		)
+		(stroke
+			(width 0)
+			(type default)
+		)
+	)
+	(wire
+		(pts
+			(xy 207.01 46.99) (xy 207.01 55.88)
 		)
 		(stroke
@@
 	(wire
 		(pts
-			(xy 74.93 54.61) (xy 86.36 54.61)
-		)
-		(stroke
-			(width 0)
-			(type default)
-		)
-	)
-	(wire
-		(pts
 			(xy 195.58 62.23) (xy 201.93 62.23)
 		)
@@
 	(wire
 		(pts
-			(xy 201.93 34.29) (xy 201.93 55.88)
-		)
-		(stroke
-			(width 0)
-			(type default)
-		)
-	)
-	(wire
-		(pts
 			(xy 68.58 63.5) (xy 71.12 63.5)
 		)
@@
 		)
 	)
-	(wire
-		(pts
-			(xy 74.93 33.02) (xy 74.93 54.61)
-		)
-		(stroke
-			(width 0)
-			(type default)
-		)
-	)
 	(polyline
 		(pts
-			(xy 180.34 171.45) (xy 180.34 99.06)
+			(xy 180.34 171.45) (xy 180.34 102.87)
 		)
 		(stroke
@@
 	(wire
 		(pts
+			(xy 74.93 52.07) (xy 86.36 52.07)
+		)
+		(stroke
+			(width 0)
+			(type default)
+		)
+	)
+	(wire
+		(pts
 			(xy 218.44 161.29) (xy 218.44 162.56)
 		)
@@
 	(wire
 		(pts
+			(xy 96.52 52.07) (xy 99.06 52.07)
+		)
+		(stroke
+			(width 0)
+			(type default)
+		)
+	)
+	(wire
+		(pts
 			(xy 180.34 73.66) (xy 180.34 74.93)
 		)
@@
 	(wire
 		(pts
-			(xy 80.01 45.72) (xy 80.01 52.07)
-		)
-		(stroke
-			(width 0)
-			(type default)
-		)
-	)
-	(wire
-		(pts
-			(xy 80.01 52.07) (xy 86.36 52.07)
+			(xy 74.93 33.02) (xy 74.93 52.07)
 		)
 		(stroke
@@
 	(wire
 		(pts
+			(xy 207.01 55.88) (xy 213.36 55.88)
+		)
+		(stroke
+			(width 0)
+			(type default)
+		)
+	)
+	(wire
+		(pts
 			(xy 66.04 139.7) (xy 67.31 139.7)
 		)
@@
 	(wire
 		(pts
-			(xy 201.93 55.88) (xy 213.36 55.88)
-		)
-		(stroke
-			(width 0)
-			(type default)
-		)
-	)
-	(wire
-		(pts
 			(xy 87.63 132.08) (xy 91.44 132.08)
 		)
@@
 		(pts
 			(xy 69.85 41.91) (xy 69.85 43.18)
-		)
-		(stroke
-			(width 0)
-			(type default)
-		)
-	)
-	(wire
-		(pts
-			(xy 207.01 46.99) (xy 207.01 53.34)
-		)
-		(stroke
-			(width 0)
-			(type default)
-		)
-	)
-	(wire
-		(pts
-			(xy 96.52 52.07) (xy 99.06 52.07)
 		)
 		(stroke
@@
 			(font
 				(size 3 3)
+			)
+			(justify left bottom)
+		)
+	)
+	(text "USB Track Impedance: Differential Pair\nhttps://saturnpcb.com/saturn-pcb-toolkit/\nPrepreg thickness: 8.3 mil (JLC7628). Er = 4.6\n10.5 mil track with 9.5 mil gap (20 mil center to center) = 90 Ohms"
+		(exclude_from_sim no)
+		(at 16.51 99.06 0)
+		(effects
+			(font
+				(size 1.27 1.27)
 			)
 			(justify left bottom)
@@
 		(lib_id "SparkFun-Coil:USB_Transformer")
 		(at 91.44 53.34 0)
+		(mirror x)
 		(unit 1)
 		(exclude_from_sim no)
@@
 		)
 		(property "Footprint" "SparkFun-Coil:RFCMF1220100M4T"
-			(at 90.17 59.69 0)
+			(at 90.17 46.99 0)
 			(effects
 				(font
@@
 		)
 		(property "Datasheet" "http://www.passivecomponent.com/wp-content/uploads/2018/10/RF-Filter.pdf"
-			(at 90.17 62.23 0)
+			(at 90.17 44.45 0)
 			(effects
 				(font
@@
 		)
 		(property "PROD_ID" "COMP-19495"
-			(at 90.17 64.77 0)
-			(effects
-				(font
+			(at 90.17 41.91 0)
+			(effects
+				(font
