File: Hardware/USB.kicad_sch (KiCad schematic)
At the start: 31 parts, among them J2 USB_C_Receptacle, J4 USB_C_Receptacle, Q1 MBT3904DW1, SW1 PTH_RA_h7.5mm, SW2 PTH_RA_h7.5mm, SW3 PTH_RA_h7.5mm, U3 CH340C

Commit message: PCB symbol updates
Connections:
- net at J2.A8 (NC): no longer J2.B8 (NC)
- net at J4.A8 (NC): no longer J4.B8 (NC)
- now unconnected: J2.NC1 (NC), J2.NC2 (NC), J2.NC3 (NC), J4.NC1 (NC), J4.NC2 (NC), J4.NC3 (NC)

Commit message: Updates for v1.0 PCB
Other:
- title: (none) -> USB
Changed lines of the file:
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@@
 	(generator_version "8.0")
 	(paper "USLetter")
+	(title_block
+		(title "USB")
+	)
 	(junction
 		(at 91.44 129.54)

Commit message: Final tweaks
Parts:
- added TP46, TP47, TP49, TP50: PTH, SparkFun-Connector:1x01, symbol SparkFun-Connector:TestPoint_PTH
Connections:
- net GND: now also TP49.1, TP50.1
- net VUSB: now also TP46.1
- net VUSB2: now also TP47.1
Other:
- note added: "Provides 5V 2A for optional TCXO"
