File: Hardware/Power.kicad_sch (KiCad schematic)
At the start: 15 parts, among them U11 AP2112K-3.3, U5 AP2112K-3.3

Commit message: More WIP
Parts:
- added C32, C36: 100uF, SparkFun-Capacitor:PANASONIC_D, symbol SparkFun-Capacitor:100uF_6.6x6.6_25V_20%
- added C33, C34, C37, C38: 10uF, SparkFun-Capacitor:C_0603_1608Metric, symbol SparkFun-Capacitor:10uF_0603_10V_20%
- added C35: 47uF, SparkFun-Capacitor:PANASONIC_D, symbol SparkFun-Capacitor:47uF_6.6x6.6_50V_20%
- added D10, D9: BAT60A, SparkFun-Semiconductor-Standard:SOD-323, symbol SparkFun-DiscreteSemi:D_Schottky_3A_10V_0.28V
- added D8: SK34A, SparkFun-Semiconductor-Standard:SMA, symbol SparkFun-DiscreteSemi:D_Schottky_3A_40V_0.55V
- added JP_POE+_1, JP_POE-_1, JP_VIN+_1, JP_VIN-_1: Measure, SparkFun-Jumper:Jumper_2_PTH_SMD_Combo-NC, symbol SparkFun-Jumper:Jumper_Measure
- added JP_POE_1: ~, SparkFun-Jumper:Jumper_2_NC_Trace, symbol SparkFun-Jumper:SolderJumper_2_Bridged
- added L3, L4: 4.7uH, SparkFun-Coil:1008_2520Metric, symbol SparkFun-Coil:4.7uH_1008_1.4A
- added R36: 49.9, SparkFun-Resistor:R_1206_3216Metric, symbol SparkFun-Resistor:49.9_1206
- added TP_VDC_1, TP_VPOE_1: PTH, SparkFun-Connector:1x01, symbol SparkFun-Connector:TestPoint_PTH
- added U6: REC15E-2405SZ, SparkFun-Semiconductor-Standard:REC15E, symbol SparkFun-IC-Power:REC15E-2405SZ
- added U7: Ag9905M, SparkFun-Semiconductor-Standard:Ag9900M, symbol SparkFun-IC-Power:Ag9905M
- renumbered TP_3V3P1 to TP_3V3P_1, TP_5V1 to TP_5V_1, TP_GND1 to TP_GND_1
Connections:
- net GND: now also C32.2, C33.2, C34.2, C36.2, C37.2, C38.2, R36.1, U6.4 (VOUT-), U7.3 (VOUT-)
- net POE+: now also JP_POE+_1.1 (A)
- net POE-: now also JP_POE-_1.1 (A)
- net at D4.C, D5.C, JP_MEAS1.1 (A): now also D10.C, D9.C
- new net: C35.1, D8.C, U6.1 (VIN+)
- new net: C35.2, JP_VIN-_1.2 (B), U6.2 (VIN-)
- new net: C36.1, C37.1, JP_POE_1.2 (B), L4.1, U7.1 (VOUT+), U7.2 (VOUT+)
- new net: C32.1, C33.1, L3.1, U6.6 (VOUT+)
- new net: D8.A, JP_VIN+_1.2 (B)
- new net: JP_POE_1.1 (A), R36.2
- new net DC_IN+: JP_VIN+_1.1 (A)
- new net DC_IN-: JP_VIN-_1.1 (A)
- new net VIN+: JP_POE+_1.2 (B), U7.5 (VIN+), U7.6 (VIN+)
- new net VIN-: JP_POE-_1.2 (B), U7.7 (VIN-), U7.8 (VIN-)
- new net VIN_DC: C34.1, D9.A, L3.2, TP_VDC_1.1
- new net VIN_POE: C38.1, D10.A, L4.2, TP_VPOE_1.1
Other:
- note added: "DC Power In"
- moved on the sheet: C20, C21, C22, C7, TP_3V3, TP_3V3P_1, TP_5V_1, TP_GND_1, U11, U5

Commit message: More WIP
Parts:
- renumbered JP_VIN+_1 to JP2, JP_VIN-_1 to JP3, JP_POE+_1 to JP4, JP_POE-_1 to JP5, JP_MEAS1 to JP6, JP_POE_1 to JP7, TP_VDC_1 to TP2, TP_VPOE_1 to TP3, TP_5V_1 to TP4, TP_3V3 to TP5, TP_GND_1 to TP6, TP_3V3P_1 to TP7
Changed lines of the file:
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@@
 		(on_board yes)
 		(dnp no)
-		(property "Reference" "JP_POE-_1"
+		(property "Reference" "JP5"
 			(at 34.29 92.71 0)
 			(effects
@@
 			(project "SparkFun_RTK_mosaic-T"
 				(path "/e3dd3ae4-244d-4cba-9cca-5d2abf83f29a/476b4701-5340-4853-910a-2af933cad777"
-					(reference "JP_POE-_1")
+					(reference "JP5")
 					(unit 1)
 				)
@@
 		(on_board yes)
 		(dnp no)
-		(property "Reference" "TP_3V3P_1"
+		(property "Reference" "TP7"
 			(at 189.23 143.51 0)
 			(effects
@@
 			(project "SparkFun_RTK_Facet_mosaic"
 				(path "/e3dd3ae4-244d-4cba-9cca-5d2abf83f29a/476b4701-5340-4853-910a-2af933cad777"
-					(reference "TP_3V3P_1")
+					(reference "TP7")
 					(unit 1)
 				)
@@
 		(dnp no)
 		(fields_autoplaced yes)
-		(property "Reference" "JP_MEAS1"
+		(property "Reference" "JP6"
 			(at 39.37 128.27 0)
 			(effects
@@
 			(project ""
 				(path "/e3dd3ae4-244d-4cba-9cca-5d2abf83f29a/476b4701-5340-4853-910a-2af933cad777"
-					(reference "JP_MEAS1")
+					(reference "JP6")
 					(unit 1)
 				)
@@
 		(dnp no)
 		(fields_autoplaced yes)
-		(property "Reference" "TP_5V_1"
+		(property "Reference" "TP4"
 			(at 76.2 143.0019 0)
 			(effects
@@
 			(project "SparkFun_RTK_Facet_mosaic"
 				(path "/e3dd3ae4-244d-4cba-9cca-5d2abf83f29a/476b4701-5340-4853-910a-2af933cad777"
-					(reference "TP_5V_1")
+					(reference "TP4")
 					(unit 1)
 				)
@@
 		(dnp no)
 		(fields_autoplaced yes)
-		(property "Reference" "TP_GND_1"
+		(property "Reference" "TP6"
 			(at 125.73 146.5579 0)
 			(effects
@@
 			(project "SparkFun_RTK_Facet_mosaic"
 				(path "/e3dd3ae4-244d-4cba-9cca-5d2abf83f29a/476b4701-5340-4853-910a-2af933cad777"
-					(reference "TP_GND_1")
+					(reference "TP6")
 					(unit 1)
 				)
@@
 		(on_board yes)
 		(dnp no)
-		(property "Reference" "JP_VIN-_1"
+		(property "Reference" "JP3"
 			(at 33.02 53.34 0)
 			(effects
@@
 			(project "SparkFun_RTK_mosaic-T"
 				(path "/e3dd3ae4-244d-4cba-9cca-5d2abf83f29a/476b4701-5340-4853-910a-2af933cad777"
-					(reference "JP_VIN-_1")
+					(reference "JP3")
 					(unit 1)
 				)
@@
 		(dnp no)
 		(fields_autoplaced yes)
-		(property "Reference" "TP_3V3"
+		(property "Reference" "TP5"
 			(at 125.73 141.7319 0)
 			(effects
@@
 			(project "SparkFun_RTK_Facet_mosaic"
 				(path "/e3dd3ae4-244d-4cba-9cca-5d2abf83f29a/476b4701-5340-4853-910a-2af933cad777"
-					(reference "TP_3V3")
+					(reference "TP5")
 					(unit 1)
 				)
@@
 		(dnp no)
 		(fields_autoplaced yes)
-		(property "Reference" "JP_VIN+_1"
+		(property "Reference" "JP2"
 			(at 33.02 30.48 0)
 			(effects
@@
 			(project ""
 				(path "/e3dd3ae4-244d-4cba-9cca-5d2abf83f29a/476b4701-5340-4853-910a-2af933cad777"
-					(reference "JP_VIN+_1")
+					(reference "JP2")
 					(unit 1)
 				)
@@
 		(dnp no)
 		(fields_autoplaced yes)
-		(property "Reference" "TP_VDC_1"
+		(property "Reference" "TP2"
 			(at 125.73 36.8299 90)
 			(effects
@@
 			(project "SparkFun_RTK_mosaic-T"
 				(path "/e3dd3ae4-244d-4cba-9cca-5d2abf83f29a/476b4701-5340-4853-910a-2af933cad777"
-					(reference "TP_VDC_1")
+					(reference "TP2")
 					(unit 1)
 				)
@@
 		(dnp no)
 		(fields_autoplaced yes)
-		(property "Reference" "TP_VPOE_1"
+		(property "Reference" "TP3"
 			(at 123.19 81.2799 90)
 			(effects
@@
 			(project "SparkFun_RTK_mosaic-T"
 				(path "/e3dd3ae4-244d-4cba-9cca-5d2abf83f29a/476b4701-5340-4853-910a-2af933cad777"
-					(reference "TP_VPOE_1")
+					(reference "TP3")
 					(unit 1)
 				)
@@
 		(dnp no)
 		(fields_autoplaced yes)
-		(property "Reference" "JP_POE_1"
+		(property "Reference" "JP7"
 			(at 90.17 85.7249 90)
 			(effects
@@
 			(project ""
 				(path "/e3dd3ae4-244d-4cba-9cca-5d2abf83f29a/476b4701-5340-4853-910a-2af933cad777"
-					(reference "JP_POE_1")
+					(reference "JP7")
 					(unit 1)
 				)
@@
 		(dnp no)
 		(fields_autoplaced yes)
-		(property "Reference" "JP_POE+_1"
+		(property "Reference" "JP4"
 			(at 34.29 74.93 0)
 			(effects
@@
 			(project "SparkFun_RTK_mosaic-T"
 				(path "/e3dd3ae4-244d-4cba-9cca-5d2abf83f29a/476b4701-5340-4853-910a-2af933cad777"
-					(reference "JP_POE+_1")
+					(reference "JP4")
 					(unit 1)
 				)

Commit message: More WIP
Changed lines of the file:
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@@
+	(polyline
+		(pts
+			(xy 137.16 59.69) (xy 12.7 59.69)
+		)
+		(stroke
+			(width 0)
+			(type dash)
+		)
+	)
 	(polyline
 		(pts

Commit message: More WIP
Other:
- moved on the sheet: C20, C21, C22, C36, C37, C38, C6, C7, D10, D4, D5, D9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

Commit message: Ready for airwire review
Changed lines of the file:
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@@
 		(fields_autoplaced yes)
 		(property "Reference" "C33"
-			(at 107.95 40.6399 0)
+			(at 107.95 39.3699 0)
 			(effects
 				(font
@@
 		)
 		(property "Value" "10uF"
-			(at 107.95 43.1799 0)
+			(at 107.95 41.9099 0)
 			(effects
 				(font
@@
 		)
 		(property "Voltage" "10V"
-			(at 107.95 43.1799 0)
+			(at 107.95 44.4499 0)
 			(effects
 				(font
@@
 				)
 				(justify left)
-				(hide yes)
 			)
 		)
@@
 		(fields_autoplaced yes)
 		(property "Reference" "C38"
-			(at 247.65 40.6399 0)
+			(at 247.65 39.3699 0)
 			(effects
 				(font
@@
 		)
 		(property "Value" "10uF"
-			(at 247.65 43.1799 0)
+			(at 247.65 41.9099 0)
 			(effects
 				(font
@@
 		)
 		(property "Voltage" "10V"
-			(at 247.65 43.1799 0)
+			(at 247.65 44.4499 0)
 			(effects
 				(font
@@
 				)
 				(justify left)
-				(hide yes)
 			)
 		)
@@
 		(fields_autoplaced yes)
 		(property "Reference" "C20"
-			(at 91.44 99.0599 0)
+			(at 91.44 97.7899 0)
 			(effects
 				(font
@@
 		)
 		(property "Value" "1.0uF"
-			(at 91.44 101.5999 0)
+			(at 91.44 100.3299 0)
 			(effects
 				(font
@@
 		)
 		(property "Voltage" "16V"
-			(at 91.44 101.5999 0)
+			(at 91.44 102.8699 0)
 			(effects
 				(font
@@
 				)
 				(justify left)
-				(hide yes)
 			)
 		)
@@
 		(fields_autoplaced yes)
 		(property "Reference" "C34"
-			(at 120.65 40.6399 0)
+			(at 120.65 39.3699 0)
 			(effects
 				(font
@@
 		)
 		(property "Value" "10uF"
-			(at 120.65 43.1799 0)
+			(at 120.65 41.9099 0)
 			(effects
 				(font
@@
 		)
 		(property "Voltage" "10V"
-			(at 120.65 43.1799 0)
+			(at 120.65 44.4499 0)
 			(effects
 				(font
@@
 				)
 				(justify left)
-				(hide yes)
 			)
 		)
@@
 		(fields_autoplaced yes)
 		(property "Reference" "C7"
-			(at 154.94 99.0599 0)
+			(at 147.32 97.7899 0)
 			(effects
 				(font
 					(size 1.27 1.27)
 				)
-				(justify left)
+				(justify right)
 			)
 		)
 		(property "Value" "1.0uF"
-			(at 154.94 101.5999 0)
+			(at 147.32 100.3299 0)
 			(effects
 				(font
 					(size 1.27 1.27)
 				)
-				(justify left)
+				(justify right)
 			)
 		)
@@
 		)
 		(property "Voltage" "16V"
-			(at 154.94 101.5999 0)
+			(at 147.32 102.8699 0)
 			(effects
 				(font
 					(size 1.27 1.27)
 				)
-				(justify left)
-				(hide yes)
+				(justify right)
 			)
 		)
@@
 		(fields_autoplaced yes)
 		(property "Reference" "C37"
-			(at 234.95 40.6399 0)
+			(at 234.95 39.3699 0)
 			(effects
 				(font
@@
 		)
 		(property "Value" "10uF"
-			(at 234.95 43.1799 0)
+			(at 234.95 41.9099 0)
 			(effects
 				(font
@@
 		)
 		(property "Voltage" "10V"
-			(at 234.95 43.1799 0)
+			(at 234.95 44.4499 0)
 			(effects
 				(font
@@
 				)
 				(justify left)
-				(hide yes)
 			)
 		)

Commit message: Updates to match latest KiCad library
Parts:
- C32, C35, C36, C6: footprint SparkFun-Capacitor:PANASONIC_D -> SparkFun-Capacitor:Panasonic_D
- U6: footprint SparkFun-Semiconductor-Standard:REC15E -> SparkFun-Semiconductor-Nonstandard:REC15E
- U7: footprint SparkFun-Semiconductor-Standard:Ag9900M -> SparkFun-Semiconductor-Nonstandard:Ag9900M
Changed lines of the file:
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@@
 			)
 		)
-		(property "Footprint" "SparkFun-Capacitor:PANASONIC_D"
+		(property "Footprint" "SparkFun-Capacitor:Panasonic_D"
 			(at 46.99 59.69 0)
 			(effects
@@
 			)
 		)
-		(property "Footprint" "SparkFun-Semiconductor-Standard:Ag9900M"
+		(property "Footprint" "SparkFun-Semiconductor-Nonstandard:Ag9900M"
 			(at 184.15 57.4675 0)
 			(effects
@@
 			)
 		)
-		(property "Footprint" "SparkFun-Semiconductor-Standard:REC15E"
+		(property "Footprint" "SparkFun-Semiconductor-Nonstandard:REC15E"
 			(at 71.12 57.4675 0)
 			(effects
@@
 			)
 		)
-		(property "Footprint" "SparkFun-Capacitor:PANASONIC_D"
+		(property "Footprint" "SparkFun-Capacitor:Panasonic_D"
 			(at 63.5 114.3 0)
 			(effects
@@
 			)
 		)
-		(property "Footprint" "SparkFun-Capacitor:PANASONIC_D"
+		(property "Footprint" "SparkFun-Capacitor:Panasonic_D"
 			(at 91.44 59.69 0)
 			(effects
@@
 			)
 		)
-		(property "Footprint" "SparkFun-Capacitor:PANASONIC_D"
+		(property "Footprint" "SparkFun-Capacitor:Panasonic_D"
 			(at 204.47 59.69 0)
 			(effects
