File: Hardware/GNSS.kicad_sch (KiCad schematic)
At the start: 47 parts, among them J1 SMA_Edge, J6 microSD, U13 SiT5358AI-FS033IT-10.000000, U2 mosaic-T

Commit message: PCB symbol updates
Parts:
- D1: value PESD0402 -> PESD0402
Changed lines of the file:
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@@
 			)
 		)
-		(property "Value" " PESD0402"
+		(property "Value" "PESD0402"
 			(at 210.82 44.45 90)
 			(effects
@@
 			)
 		)
-		(property "Datasheet" "https://datasheet.lcsc.com/lcsc/2110151630_XKB-Connectivity-XKTF-015-N_C381082.pdf"
+		(property "Datasheet" "https://cdn.sparkfun.com/assets/a/d/6/0/8/microSD_Datasheet_msd-1-a.pdf"
 			(at 82.55 203.2 0)
 			(effects

Commit message: Updates for v1.0 PCB
Parts:
- added C73: 2.2uF, SparkFun-Capacitor:C_0603_1608Metric, symbol SparkFun-Capacitor:2.2uF_0603_10V_20%
- added C74: 0.1uF, SparkFun-Capacitor:C_0603_1608Metric, symbol SparkFun-Capacitor:0.1uF_0603_25V_20%
- added TP41: PTH, SparkFun-Connector:1x01, symbol SparkFun-Connector:TestPoint_PTH
Connections:
- net GND: now also C73.2, C74.2
- net ESP23/MRX3: now reaches TP16.1, U2.K1 (COM3_RX)
- net ESP34/MTX3: now reaches TP17.1, U2.M1 (COM3_TX)
- net 2.8V: now reaches U2.N23 (2V8_OUT)
- net 2.8V: now also C73.1, C74.1, TP41.1
Other:
- note added: "Console access (via TCP)"
- title: (none) -> GNSS
- moved on the sheet: C16, C17, C18, C19, C29, R5, TP16, TP17, TP18, TP19, TP22, TP29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

Commit message: Add mounting holes for SiT5811 / Rakon oscillator
Parts:
- removed R51: 0, SparkFun-Resistor:R_0603_1608Metric, symbol SparkFun-Resistor:0_0603
- added U.1: ~, SparkFun-Jumper:Jumper_2_NC_Trace, symbol SparkFun-Jumper:SolderJumper_2_Bridged
Connections:
- net 10MHz: now also U.1.2 (B)
- net at U13.6 (CLK): now also U.1.1 (A)
Other:
- note added: "Open jumper U to isolate 10MHz"
Changed lines of the file:
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@@
 		)
 	)
+	(text "Open jumper U\nto isolate 10MHz"
+		(exclude_from_sim no)
+		(at 234.95 118.11 0)
+		(effects
+			(font
+				(size 1.27 1.27)
+			)
+			(justify left)
+		)
+	)
 	(text "mosaic Tri-band GNSS\n"
 		(exclude_from_sim no)
@@
 	)
 	(symbol
+		(lib_id "SparkFun-Jumper:SolderJumper_2_Bridged")
+		(at 226.06 123.19 0)
+		(unit 1)
+		(exclude_from_sim no)
+		(in_bom yes)
+		(on_board yes)
+		(dnp no)
+		(property "Reference" "U.1"
+			(at 226.06 120.65 0)
+			(effects
+				(font
+					(size 1.27 1.27)
+				)
+			)
+		)
+		(property "Value" "~"
+			(at 226.06 120.65 0)
+			(effects
+				(font
+					(size 1.27 1.27)
+				)
+			)
+		)
+		(property "Footprint" "SparkFun-Jumper:Jumper_2_NC_Trace"
+			(at 225.806 127.762 0)
+			(effects
+				(font
+					(size 1.27 1.27)
+				)
+				(hide yes)
+			)
+		)
+		(property "Datasheet" "~"
+			(at 226.06 130.81 0)
+			(effects
+				(font
+					(size 1.27 1.27)
+				)
+				(hide yes)
+			)
+		)
+		(property "Description" "Solder Jumper, 2-pole, closed/bridged"
+			(at 226.06 133.35 0)
+			(effects
+				(font
+					(size 1.27 1.27)
+				)
+				(hide yes)
+			)
+		)
+		(pin "1"
+		)
+		(pin "2"
+		)
+		(instances
+			(project ""
+				(path "/e3dd3ae4-244d-4cba-9cca-5d2abf83f29a/1004b21d-c362-4c5d-adad-4952c3ff3811"
+					(reference "U.1")
+					(unit 1)
+				)
+			)
+		)
+	)
+	(symbol
 		(lib_id "SparkFun-Connector:TestPoint_PTH")
 		(at 59.69 109.22 90)
@@
 					(unit 1)
 				)
-			)
-		)
-	)
-	(symbol
-		(lib_id "SparkFun-Resistor:0_0603")
-		(at 226.06 123.19 0)
-		(unit 1)
-		(exclude_from_sim no)
-		(in_bom yes)
-		(on_board yes)
-		(dnp no)
-		(fields_autoplaced yes)
-		(property "Reference" "R51"
-			(at 226.06 116.84 0)
-			(effects
-				(font
-					(size 1.27 1.27)
-				)
-			)
-		)
-		(property "Value" "0"
-			(at 226.06 119.38 0)
-			(effects
-				(font
-					(size 1.27 1.27)
-				)
-			)
-		)
-		(property "Footprint" "SparkFun-Resistor:R_0603_1608Metric"
-			(at 226.06 127.762 0)
-			(effects
-				(font
-					(size 1.27 1.27)
-				)
-				(hide yes)
-			)
-		)
-		(property "Datasheet" "https://industrial.panasonic.com/cdbs/www-data/pdf/RDN0000/AOA0000C313.pdf"
-			(at 226.06 132.08 0)
-			(effects
-				(font
-					(size 1.27 1.27)
-				)
-				(hide yes)
-			)
-		)
-		(property "Description" "Resistor"
-			(at 226.06 134.62 0)
-			(effects
-				(font
-					(size 1.27 1.27)
-				)
-				(hide yes)
-			)
-		)
-		(property "PROD_ID" "RES-08609"
-			(at 226.06 130.048 0)
-			(effects
-				(font
-					(size 1.27 1.27)
-				)
-				(hide yes)
-			)
-		)
-		(pin "2"
-		)
-		(pin "1"
-		)
-		(instances
-			(project "SparkFun_RTK_mosaic-T"
-				(path "/e3dd3ae4-244d-4cba-9cca-5d2abf83f29a/1004b21d-c362-4c5d-adad-4952c3ff3811"
-					(reference "R51")
-					(unit 1)
-				)

Commit message: Final changes before name change
Connections:
- net 5V is gone; now on net 3.3V_P: L1.1
Other:
- note added: "I/O Screw Terminal (via level-shifter)"
- note added: "SMA Connectors (via level-shifters)"
Changed lines of the file:
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@@
 		)
 	)
-	(polyline
-		(pts
-			(xy 115.57 96.52) (xy 115.57 99.06)
-		)
-		(stroke
-			(width 0)
-			(type default)
-		)
-	)
 	(wire
 		(pts
@@
 	(polyline
 		(pts
-			(xy 115.57 101.6) (xy 115.57 104.14)
+			(xy 115.57 100.33) (xy 115.57 101.6)
 		)
 		(stroke
@@
 		)
 	)
+	(polyline
+		(pts
+			(xy 115.57 96.52) (xy 115.57 97.79)
+		)
+		(stroke
+			(width 0)
+			(type default)
+		)
+	)
 	(wire
 		(pts
@@
 	)
 	(arc
-		(start 116.84 100.33)
-		(mid 115.942 99.958)
-		(end 115.57 99.06)
+		(start 116.84 99.06)
+		(mid 115.942 98.688)
+		(end 115.57 97.79)
 		(stroke
 			(width 0)
@@
 	)
 	(arc
-		(start 115.57 101.6)
-		(mid 115.942 100.702)
-		(end 116.84 100.33)
+		(start 115.57 100.33)
+		(mid 115.942 99.432)
+		(end 116.84 99.06)
 		(stroke
 			(width 0)
@@
 	)
 	(arc
-		(start 115.57 104.14)
-		(mid 115.198 105.038)
-		(end 114.3 105.41)
+		(start 115.57 101.6)
+		(mid 115.198 102.498)
+		(end 114.3 102.87)
 		(stroke
 			(width 0)
@@
 		)
 	)
-	(text "I/O Screw Terminals\n(via level-shifters)"
+	(text "SMA Connectors\n(via level-shifters)"
 		(exclude_from_sim no)
-		(at 118.11 101.6 0)
+		(at 125.73 101.6 0)
 		(effects
 			(font
 				(size 1.27 1.27)
 			)
-			(justify left bottom)
+			(justify bottom)
 		)
 	)
@@
 		)
 	)
+	(text "I/O Screw Terminal\n(via level-shifter)"
+		(exclude_from_sim no)
+		(at 125.73 107.95 0)
+		(effects
+			(font
+				(size 1.27 1.27)
+			)
+			(justify bottom)
+		)
+	)
 	(text "50MHz"
 		(exclude_from_sim no)
@@
 	)
 	(symbol
-		(lib_id "SparkFun-PowerSymbol:5V")
-		(at 43.18 45.72 0)
-		(unit 1)
-		(exclude_from_sim no)
-		(in_bom yes)
-		(on_board yes)
-		(dnp no)
-		(fields_autoplaced yes)
-		(property "Reference" "#PWR08"
-			(at 43.18 49.53 0)
-			(effects
-				(font
-					(size 1.27 1.27)
-				)
-				(hide yes)
-			)
-		)
-		(property "Value" "5V"
-			(at 43.18 41.91 0)
-			(do_not_autoplace yes)
-			(effects
-				(font
-					(size 1.27 1.27)
-				)
-			)
-		)
-		(property "Footprint" ""
-			(at 43.18 45.72 0)
-			(effects
-				(font
-					(size 1.27 1.27)
-				)
-				(hide yes)
-			)
-		)
-		(property "Datasheet" ""
-			(at 43.18 45.72 0)
-			(effects
-				(font
-					(size 1.27 1.27)
-				)
-				(hide yes)
-			)
-		)
-		(property "Description" "Power symbol creates a global label with name \"5V\""
-			(at 43.18 45.72 0)
-			(effects
-				(font
-					(size 1.27 1.27)
-				)
-				(hide yes)
-			)
-		)
-		(pin "1"
-		)
-		(instances
-			(project "SparkFun_RTK_mosaic-T"
-				(path "/e3dd3ae4-244d-4cba-9cca-5d2abf83f29a/1004b21d-c362-4c5d-adad-4952c3ff3811"
-					(reference "#PWR08")
-					(unit 1)
-				)
-			)
-		)
-	)
-	(symbol
 		(lib_id "SparkFun-DiscreteSemi:D_TVS_ESD_4_HS")
 		(at 60.96 187.96 0)
@@
 					(unit 1)
 				)
+			)
+		)
+	)
+	(symbol
+		(lib_id "SparkFun-PowerSymbol:3.3V_P")
+		(at 43.18 45.72 0)
+		(unit 1)
+		(exclude_from_sim no)
+		(in_bom yes)
+		(on_board yes)
+		(dnp no)
+		(property "Reference" "#PWR08"
+			(at 43.18 49.53 0)
+			(effects
+				(font
+					(size 1.27 1.27)
+				)
+				(hide yes)
+			)
+		)
+		(property "Value" "3.3V_P"
+			(at 43.18 41.91 0)
+			(effects
+				(font
+					(size 1.27 1.27)
+				)
+			)
+		)
+		(property "Footprint" ""
+			(at 43.18 45.72 0)
+			(effects
+				(font
+					(size 1.27 1.27)
+				)
+				(hide yes)
+			)
+		)
+		(property "Datasheet" ""
+			(at 43.18 45.72 0)
+			(effects
+				(font
+					(size 1.27 1.27)
+				)
+				(hide yes)
+			)
+		)
+		(property "Description" "Power symbol creates a global label with name \"3.3V_P\""
+			(at 43.18 45.72 0)
+			(effects
+				(font
+					(size 1.27 1.27)
+				)
+				(hide yes)
+			)
+		)
+		(pin "1"
+		)
+		(instances
+			(project "SparkFun_RTK_mosaic-T"
+				(path "/e3dd3ae4-244d-4cba-9cca-5d2abf83f29a/1004b21d-c362-4c5d-adad-4952c3ff3811"
+					(reference "#PWR08")
+					(unit 1)
+				)
