File: Hardware/SparkPNT_GPSDO.kicad_sch (KiCad schematic)
At the start: 49 parts, among them J7 Qwiic_Vertical, J9 Screw_Cage_3.5mm-10, U1 ESP32-WROVER-IE-N16R8

Commit message: Rename to GNSSDO
Other:
- title: GPSDO (mosaic-T, SiT5358) -> GNSSDO (mosaic-T, SiT5358)
Changed lines of the file:
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@@
 	(paper "USLetter")
 	(title_block
-		(title "GPSDO (mosaic-T, SiT5358)")
+		(title "GNSSDO (mosaic-T, SiT5358)")
 		(date "2024-11-08")
 		(rev "v10")
@@
 		)
 		(instances
-			(project "SparkPNT_GPSDO"
+			(project "SparkPNT_GNSSDO"
 				(path "/e3dd3ae4-244d-4cba-9cca-5d2abf83f29a"
 					(page "3")
@@
 		)
 		(instances
-			(project "SparkPNT_GPSDO"
+			(project "SparkPNT_GNSSDO"
 				(path "/e3dd3ae4-244d-4cba-9cca-5d2abf83f29a"
 					(page "4")
@@
 		)
 		(instances
-			(project "SparkPNT_GPSDO"
+			(project "SparkPNT_GNSSDO"
 				(path "/e3dd3ae4-244d-4cba-9cca-5d2abf83f29a"
 					(page "2")
@@
 		)
 		(instances
-			(project "SparkPNT_GPSDO"
+			(project "SparkPNT_GNSSDO"
 				(path "/e3dd3ae4-244d-4cba-9cca-5d2abf83f29a"
 					(page "5")
@@
 		)
 		(instances
-			(project "SparkPNT_GPSDO"
+			(project "SparkPNT_GNSSDO"
 				(path "/e3dd3ae4-244d-4cba-9cca-5d2abf83f29a"
 					(page "6")
@@
 		)
 		(instances
-			(project "SparkPNT_GPSDO"
+			(project "SparkPNT_GNSSDO"
 				(path "/e3dd3ae4-244d-4cba-9cca-5d2abf83f29a"
 					(page "7")
