File: Hardware/GNSSDO_Plus/Level_Shifting_10MHz.kicad_sch (KiCad schematic)
At the start: 59 parts, among them J10 SMA_Edge, J8 SMA_Edge, U15 SN74LVC1G175DCK, U17 LMV7219M5, U20 LMV7219M5, U23 LMV7219M5, U24 LMV7219M5

Commit message: Update GNSSDO KiCad files to match latest SparkFun library
Parts:
- C71, C72, C80, C84: PROD_ID CAP-07888 -> CAP-24999
- J10, J8: footprint SparkFun-Connector:SMA_Edge -> SparkFun-Connector:SMA_Edge_6.3mm; symbol SparkFun-RF:SMA_EdgeMount -> SparkFun-RF:SMA_EdgeMount_6.3mm
- U15: footprint SparkFun-Semiconductor-Standard:SOT-323 -> SparkFun-Semiconductor-Standard:SOT-363_SC-70-6
Changed lines of the file:
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@@
 		)
 		(instances
-			(project "SparkFun_RTK_mosaic-T"
+			(project "SparkPNT_GNSSDO_Plus"
 				(path "/e3dd3ae4-244d-4cba-9cca-5d2abf83f29a/e788e229-99ae-40ff-993c-e79a627e85af"
 					(reference "#PWR249")
@@
 		)
 		(instances
-			(project "SparkFun_RTK_mosaic-T"
+			(project "SparkPNT_GNSSDO_Plus"
 				(path "/e3dd3ae4-244d-4cba-9cca-5d2abf83f29a/e788e229-99ae-40ff-993c-e79a627e85af"
 					(reference "#PWR247")
@@
 		)
 		(instances
-			(project "SparkFun_RTK_mosaic-T"
+			(project "SparkPNT_GNSSDO_Plus"
 				(path "/e3dd3ae4-244d-4cba-9cca-5d2abf83f29a/e788e229-99ae-40ff-993c-e79a627e85af"
 					(reference "#PWR211")
@@
 			)
 		)
-		(property "PROD_ID" "CAP-07888"
+		(property "PROD_ID" "CAP-24999"
 			(at 30.48 66.04 0)
 			(effects
@@
 		)
 		(instances
-			(project "SparkFun_RTK_mosaic-T"
+			(project "SparkPNT_GNSSDO_Plus"
 				(path "/e3dd3ae4-244d-4cba-9cca-5d2abf83f29a/e788e229-99ae-40ff-993c-e79a627e85af"
 					(reference "C71")
@@
 		)
 		(instances
-			(project "SparkFun_RTK_mosaic-T"
+			(project "SparkPNT_GNSSDO_Plus"
 				(path "/e3dd3ae4-244d-4cba-9cca-5d2abf83f29a/e788e229-99ae-40ff-993c-e79a627e85af"
 					(reference "R57")
@@
 		)
 		(instances
-			(project "SparkFun_RTK_mosaic-T"
+			(project "SparkPNT_GNSSDO_Plus"
 				(path "/e3dd3ae4-244d-4cba-9cca-5d2abf83f29a/e788e229-99ae-40ff-993c-e79a627e85af"
 					(reference "C68")
@@
 		)
 		(instances
-			(project ""
+			(project "SparkPNT_GNSSDO_Plus"
 				(path "/e3dd3ae4-244d-4cba-9cca-5d2abf83f29a/e788e229-99ae-40ff-993c-e79a627e85af"
 					(reference "R77")
@@
 			)
 		)
-		(property "Footprint" "SparkFun-Semiconductor-Standard:SOT-323"
+		(property "Footprint" "SparkFun-Semiconductor-Standard:SOT-363_SC-70-6"
 			(at 161.29 160.02 0)
 			(effects
@@
 			)
 		)
-		(property "Description" "Single D-Type Flip-Flop With Asynchronous Clear, 1.65V to 5.5V, SOT-323 (SC70)"
+		(property "Description" "Single D-Type Flip-Flop With Asynchronous Clear, 1.65V to 5.5V, SOT-363 (SC70)"
 			(at 161.29 167.64 0)
 			(effects
@@
 		)
 		(instances
-			(project ""
+			(project "SparkPNT_GNSSDO_Plus"
 				(path "/e3dd3ae4-244d-4cba-9cca-5d2abf83f29a/e788e229-99ae-40ff-993c-e79a627e85af"
 					(reference "U15")
@@
 			)
 		)
-		(property "PROD_ID" "CAP-07888"
+		(property "PROD_ID" "CAP-24999"
 			(at 30.48 179.07 0)
 			(effects
@@
 		)
 		(instances
-			(project "SparkFun_RTK_mosaic-T"
+			(project "SparkPNT_GNSSDO_Plus"
 				(path "/e3dd3ae4-244d-4cba-9cca-5d2abf83f29a/e788e229-99ae-40ff-993c-e79a627e85af"
 					(reference "D17")
@@
 		)
 		(instances
-			(project "SparkFun_RTK_mosaic-T"
+			(project "SparkPNT_GNSSDO_Plus"
 				(path "/e3dd3ae4-244d-4cba-9cca-5d2abf83f29a/e788e229-99ae-40ff-993c-e79a627e85af"
 					(reference "R50")
@@
 		)
 		(instances
-			(project "SparkFun_RTK_mosaic-T"
+			(project "SparkPNT_GNSSDO_Plus"
 				(path "/e3dd3ae4-244d-4cba-9cca-5d2abf83f29a/e788e229-99ae-40ff-993c-e79a627e85af"
 					(reference "#PWR203")
@@
 		)
 		(instances
-			(project ""
+			(project "SparkPNT_GNSSDO_Plus"
 				(path "/e3dd3ae4-244d-4cba-9cca-5d2abf83f29a/e788e229-99ae-40ff-993c-e79a627e85af"
 					(reference "TP47")
@@
 		)
 		(instances
-			(project "SparkFun_RTK_mosaic-T"
+			(project "SparkPNT_GNSSDO_Plus"
 				(path "/e3dd3ae4-244d-4cba-9cca-5d2abf83f29a/e788e229-99ae-40ff-993c-e79a627e85af"
 					(reference "#PWR256")
@@
 		)
 		(instances
-			(project "SparkFun_RTK_mosaic-T"
+			(project "SparkPNT_GNSSDO_Plus"
 				(path "/e3dd3ae4-244d-4cba-9cca-5d2abf83f29a/e788e229-99ae-40ff-993c-e79a627e85af"
 					(reference "R52")
@@
 		)
 		(instances
-			(project ""
+			(project "SparkPNT_GNSSDO_Plus"
 				(path "/e3dd3ae4-244d-4cba-9cca-5d2abf83f29a/e788e229-99ae-40ff-993c-e79a627e85af"
 					(reference "TP46")
@@
 			)
 		)
-		(property "PROD_ID" "CAP-07888"
+		(property "PROD_ID" "CAP-24999"
 			(at 30.48 44.45 0)
 			(effects
@@
 		)
 		(instances
-			(project "SparkFun_RTK_mosaic-T"
+			(project "SparkPNT_GNSSDO_Plus"
 				(path "/e3dd3ae4-244d-4cba-9cca-5d2abf83f29a/e788e229-99ae-40ff-993c-e79a627e85af"
 					(reference "C72")
@@
 		)
 		(instances
-			(project ""
+			(project "SparkPNT_GNSSDO_Plus"
 				(path "/e3dd3ae4-244d-4cba-9cca-5d2abf83f29a/e788e229-99ae-40ff-993c-e79a627e85af"
 					(reference "R76")
@@
 		)
 		(instances
-			(project "SparkFun_RTK_mosaic-T"
+			(project "SparkPNT_GNSSDO_Plus"
 				(path "/e3dd3ae4-244d-4cba-9cca-5d2abf83f29a/e788e229-99ae-40ff-993c-e79a627e85af"
 					(reference "C76")
@@
 		)
 		(instances
-			(project "SparkFun_RTK_mosaic-T"
+			(project "SparkPNT_GNSSDO_Plus"
 				(path "/e3dd3ae4-244d-4cba-9cca-5d2abf83f29a/e788e229-99ae-40ff-993c-e79a627e85af"
 					(reference "#PWR210")
@@
 		)
 		(instances
-			(project "SparkFun_RTK_mosaic-T"
+			(project "SparkPNT_GNSSDO_Plus"
 				(path "/e3dd3ae4-244d-4cba-9cca-5d2abf83f29a/e788e229-99ae-40ff-993c-e79a627e85af"
 					(reference "#PWR195")
@@
 		)
 		(instances
-			(project "SparkFun_RTK_mosaic-T"
+			(project "SparkPNT_GNSSDO_Plus"
 				(path "/e3dd3ae4-244d-4cba-9cca-5d2abf83f29a/e788e229-99ae-40ff-993c-e79a627e85af"
 					(reference "R56")
@@
 	)
 	(symbol
-		(lib_id "SparkFun-RF:SMA_EdgeMount")
+		(lib_id "SparkFun-RF:SMA_EdgeMount_6.3mm")
 		(at 166.37 34.29 0)
 		(unit 1)
@@
 			)
 		)
-		(property "Footprint" "SparkFun-Connector:SMA_Edge"
+		(property "Footprint" "SparkFun-Connector:SMA_Edge_6.3mm"
 			(at 166.37 44.45 0)
 			(effects
@@
 			)
 		)
-		(property "Datasheet" "https://www.sparkfun.com/datasheets/Wireless/Antenna/SMA-Connector.pdf"
+		(property "Datasheet" "https://cdn.sparkfun.com/assets/4/1/2/2/0/SMA-Connector.pdf"
 			(at 166.37 46.99 0)
 			(effects
@@
 			)
 		)
-		(property "Description" "SMA PCB Edge Mount connector"
+		(property "Description" "Not for new designs. Use 8mm variant. SMA PCB Edge Mount connector"
 			(at 166.37 49.53 0)
 			(effects
@@
 		)
 		(instances
-			(project "SparkFun_RTK_mosaic-T"
+			(project "SparkPNT_GNSSDO_Plus"
 				(path "/e3dd3ae4-244d-4cba-9cca-5d2abf83f29a/e788e229-99ae-40ff-993c-e79a627e85af"
 					(reference "J8")
@@
 		)
 		(instances
-			(project ""
+			(project "SparkPNT_GNSSDO_Plus"
 				(path "/e3dd3ae4-244d-4cba-9cca-5d2abf83f29a/e788e229-99ae-40ff-993c-e79a627e85af"
 					(reference "U17")
@@
 		)
 		(instances
-			(project ""
+			(project "SparkPNT_GNSSDO_Plus"
 				(path "/e3dd3ae4-244d-4cba-9cca-5d2abf83f29a/e788e229-99ae-40ff-993c-e79a627e85af"
 					(reference "C75")
@@
 		)
 		(instances
-			(project "SparkFun_RTK_mosaic-T"
+			(project "SparkPNT_GNSSDO_Plus"
 				(path "/e3dd3ae4-244d-4cba-9cca-5d2abf83f29a/e788e229-99ae-40ff-993c-e79a627e85af"
 					(reference "#PWR254")
@@
 		)
 		(instances
-			(project ""
+			(project "SparkPNT_GNSSDO_Plus"
 				(path "/e3dd3ae4-244d-4cba-9cca-5d2abf83f29a/e788e229-99ae-40ff-993c-e79a627e85af"
 					(reference "C83")
@@
 		)
 		(instances
-			(project "SparkFun_RTK_mosaic-T"
+			(project "SparkPNT_GNSSDO_Plus"
 				(path "/e3dd3ae4-244d-4cba-9cca-5d2abf83f29a/e788e229-99ae-40ff-993c-e79a627e85af"
 					(reference "#PWR252")
@@
 			)
 		)
-		(property "PROD_ID" "CAP-07888"
+		(property "PROD_ID" "CAP-24999"
 			(at 30.48 113.03 0)
 			(effects
@@
 		)
 		(instances
-			(project "SparkFun_RTK_mosaic-T"
+			(project "SparkPNT_GNSSDO_Plus"
 				(path "/e3dd3ae4-244d-4cba-9cca-5d2abf83f29a/e788e229-99ae-40ff-993c-e79a627e85af"
 					(reference "#PWR255")
@@
 	)
 	(symbol
-		(lib_id "SparkFun-RF:SMA_EdgeMount")
+		(lib_id "SparkFun-RF:SMA_EdgeMount_6.3mm")
 		(at 212.09 151.13 0)
 		(unit 1)
@@
 			)
 		)
-		(property "Footprint" "SparkFun-Connector:SMA_Edge"
+		(property "Footprint" "SparkFun-Connector:SMA_Edge_6.3mm"
 			(at 212.09 161.29 0)
 			(effects
@@
 			)
 		)
-		(property "Datasheet" "https://www.sparkfun.com/datasheets/Wireless/Antenna/SMA-Connector.pdf"
+		(property "Datasheet" "https://cdn.sparkfun.com/assets/4/1/2/2/0/SMA-Connector.pdf"
 			(at 212.09 163.83 0)
 			(effects
@@
 			)
 		)
-		(property "Description" "SMA PCB Edge Mount connector"
+		(property "Description" "Not for new designs. Use 8mm variant. SMA PCB Edge Mount connector"
 			(at 212.09 166.37 0)
 			(effects
@@
 		)
 		(instances
-			(project "SparkFun_RTK_mosaic-T"
+			(project "SparkPNT_GNSSDO_Plus"
 				(path "/e3dd3ae4-244d-4cba-9cca-5d2abf83f29a/e788e229-99ae-40ff-993c-e79a627e85af"
 					(reference "#PWR202")
@@
 		)
 		(instances
-			(project "SparkFun_RTK_mosaic-T"
+			(project "SparkPNT_GNSSDO_Plus"
 				(path "/e3dd3ae4-244d-4cba-9cca-5d2abf83f29a/e788e229-99ae-40ff-993c-e79a627e85af"
 					(reference "C69")
@@
 		)
 		(instances
-			(project "SparkFun_RTK_mosaic-T"
+			(project "SparkPNT_GNSSDO_Plus"
 				(path "/e3dd3ae4-244d-4cba-9cca-5d2abf83f29a/e788e229-99ae-40ff-993c-e79a627e85af"
 					(reference "#PWR248")
@@
 		)
 		(instances
-			(project "SparkFun_RTK_mosaic-T"
+			(project "SparkPNT_GNSSDO_Plus"
 				(path "/e3dd3ae4-244d-4cba-9cca-5d2abf83f29a/e788e229-99ae-40ff-993c-e79a627e85af"
 					(reference "C70")
@@
 		)
 		(instances
-			(project "SparkFun_RTK_mosaic-T"
+			(project "SparkPNT_GNSSDO_Plus"
 				(path "/e3dd3ae4-244d-4cba-9cca-5d2abf83f29a/e788e229-99ae-40ff-993c-e79a627e85af"
 					(reference "#PWR250")
