File: Hardware/GNSSDO_Plus/SparkPNT_GNSSDO_Plus.kicad_pcb (KiCad board)
At the start: 4 copper layers, 151.9 x 101.6 mm, 472 parts, among them J1 SMA_Edge, J10 SMA_Edge, J2 USB_C_Receptacle, J3 SMA_Edge, J4 USB_C_Receptacle, J5 MagJack_PoE, J6 microSD, J7 Qwiic_Vertical, J8 SMA_Edge, J9 Screw_Cage_3.5mm-10, Q1 MBT3904DW1, Q2 DMG2305UX, Q3 DMG2305UX, Q4 DMG2305UX, Q5 DMG2305UX, Q6 DMG2305UX, Q7 DMG2305UX, Q8 DMG2305UX, Q9 DMG2305UX, SW1 PTH_RA_h7.5mm, SW2 PTH_RA_h7.5mm, SW3 PTH_RA_h7.5mm, SW4 DPDT_Slide_SMD_7.2x3.5mm, U1 ESP32-WROVER-IE-N16R8, U10 74LVC2T45DC, U11 AP7361C-3.3V, U12 74LVC2T45DC, U13 STP3593LF, U14 74LVC2T45DC, U15 SN74LVC1G175DCK, U16 JPS-3-1+, U17 LMV7219M5, U18 MS8607-02BA, U19 PCA9306, U2 mosaic-T, U20 LMV7219M5, U23 LMV7219M5, U24 LMV7219M5, U25 AP2112K-3.3, U26 LTC4418, U27 LTC4418, U3 CH340C, U4 KSZ8041NL/I, U5 AP7361C-3.3V, U6 REC15E-2405SZ, U7 DP5305, U8 74LVC2T45DC, U9 74LVC2T45DC

Commit message: Reduce PCB width by 1.5mm. Bump to v10
Other:
- board text added: "v10"
- board text removed: "v02"
Changed lines of the file:
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@@
 		)
 	)
-	(gr_text "v02"
+	(gr_text "v10"
 		(at 104.14 132.08 270)
 		(layer "B.Cu" knockout)
