File: Hardware/GNSSDO/Power.kicad_sch (KiCad schematic)
At the start: 38 parts, among them U11 AP7361C-3.3V, U5 AP7361C-3.3V, U6 REC15E-2405SZ, U7 Ag9905M

Commit message: KiCad 10
Parts:
- JP7: value ~ -> (none)
- TP2, TP3, TP4, TP45, TP5, TP6, TP7: footprint SparkFun-Connector:1x01 -> SparkFun-Connector:1x01_P2.54mm
- U11, U5: footprint SparkFun-Semiconductor-Standard:UDFN-8 -> SparkFun-Semiconductor-Standard:DFN-8_3x3mm_P0.65mm_EP2.25x1.5mm; IMax (none) -> 1.5A
Connections:
- net 5V: now also F1.2; no longer F1.1
- net GND: now also R36.2; no longer R36.1
- net VIN_DC: now also D9.2 (A); no longer D9.A
- net VIN_POE: now also D10.2 (A); no longer D10.A
- net VUSB: now also D4.2 (A); no longer D4.A
- net VUSB2: now also D5.2 (A); no longer D5.A
- net at C35.1, U6.1 (VIN+): now also D8.1 (K); no longer D8.C
- net at JP6.2 (B): now also F1.1; no longer F1.2
- net at JP2.2 (B): now also D8.2 (A); no longer D8.A
- net at JP7.1 (A): now also R36.1; no longer R36.2
- new net: D10.1 (K), D4.1 (K), D5.1 (K), D9.1 (K), JP6.1 (A)
- now unconnected: U11.2 (NC), U11.3 (NC), U11.6 (NC), U11.7 (NC), U5.2 (NC), U5.3 (NC), U5.6 (NC), U5.7 (NC)
- no-connect marks 0 -> 3
Other:
- moved on the sheet: C22, C6, C7, JP4, JP5
