File: Hardware/GNSSDO/SparkPNT_GPSDO.kicad_pcb (KiCad board)
At the start: 4 copper layers, 151.9 x 101.6 mm, 438 parts, among them J1 SMA_Edge, J12 SMA_Edge, J2 USB_C_Receptacle, J3 SMA_Edge, J4 USB_C_Receptacle, J5 MagJack_PoE, J6 microSD, J7 Qwiic_Vertical, J8 SMA_Edge, J9 Screw_Cage_3.5mm-10, Q1 MBT3904DW1, SW1 PTH_RA_h7.5mm, SW2 PTH_RA_h7.5mm, SW3 PTH_RA_h7.5mm, SW4 DPDT_Slide_SMD_7.2x3.5mm, SW5 DPDT_Slide_SMD_7.2x3.5mm, U1 ESP32-WROVER-IE-N16R8, U10 74LVC2T45DC, U11 AP7361C-3.3V, U12 74LVC2T45DC, U13 SiT5358AI-FS033IT-10.000000, U14 74LVC2T45DC, U15 74LVC2T45DC, U16 74LVC2T45DC, U17 LMV7219M5, U18 PCA9306, U2 mosaic-T, U3 CH340C, U4 KSZ8041NL/I, U5 AP7361C-3.3V, U6 REC15E-2405SZ, U7 Ag9905M, U8 74LVC2T45DC, U9 74LVC2T45DC

Commit message: KiCad 10
Parts:
- C9: value 1nF -> 1.0nF
- J1, J12, J3, J8: footprint SparkFun-Connector:SMA_Edge -> SparkFun-Connector:SMA_Edge_6.3mm
- J7: footprint SparkFun-Connector:JST_SMD_1.0mm-4_Vertical -> SparkFun-Connector:JST_1x04_P1.0mm_Vertical_SMD
- J9: footprint SparkFun-Connector:Screw_Cage_3.5mm-10 -> SparkFun-Connector:ScrewCage_1x10_P3.5mm_Horizontal
- L1, L2: value 470Ohm -> 470 Ohm
- Q1: footprint SparkFun-Semiconductor-Standard:SOT-323 -> SparkFun-Semiconductor-Standard:SOT-363_SC-70-6
- TP1, TP10, TP11, TP12, TP13, TP14, TP15, TP16, TP17, TP18, TP19, TP2, TP20, TP21, TP22, TP23, TP24, TP25, TP26, TP27, TP28, TP29, TP3, TP30, TP31, TP32, TP33, TP34, TP35, TP36, TP37, TP38, TP39, TP4, TP40, TP41, TP42, TP43, TP44, TP45, TP46, TP47, TP48, TP49, TP5, TP50, TP6, TP7, TP8, TP9: footprint SparkFun-Connector:1x01 -> SparkFun-Connector:1x01_P2.54mm
- TR1: footprint SparkFun-Coil:RFCMF1220100M4T -> SparkFun-Coil:Choke_100MHz_USB
- U11, U5: footprint SparkFun-Semiconductor-Standard:UDFN-8 -> SparkFun-Semiconductor-Standard:DFN-8_3x3mm_P0.65mm_EP2.25x1.5mm
- U2: footprint SparkFun-GPS:MOSAIC_LGA -> SparkFun-GNSS:Septentrio_mosaic_LGA
- turned F1 to 0 degrees
- turned R1 to 180 degrees
- turned R10 to 90 degrees
- turned R11 to 90 degrees
- turned R12 to -90 degrees
- turned R13 to -90 degrees
- turned R14 to 90 degrees
- turned R15 to 90 degrees
- turned R16 to -90 degrees
- turned R17 to -90 degrees
- turned R18 to -90 degrees
- turned R19 to 180 degrees
- turned R2 to -90 degrees
- turned R20 to 180 degrees
- turned R21 to 0 degrees
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Connections:
- C35 pad 1: Net-(U6-VIN+) -> Net-(D8-K)
- C76 pad 2: Net-(U17--) -> Net-(D16-A)
- F1 pad 1: 5V -> Net-(JP6-B)
- F1 pad 2: Net-(JP6-B) -> 5V
- J6 pad 11: (no net) -> unconnected-(J6-SHIELD-Pad11)
- J6 pad 12: (no net) -> unconnected-(J6-SHIELD-Pad12)
- J6 pad 13: (no net) -> unconnected-(J6-SHIELD-Pad13)
- JP1 pad 3: Net-(JP1-B) -> Net-(JP1-C)
- JP14 pad 3: Net-(JP14-B) -> Net-(JP14-C)
- JP2 pad 2: Net-(JP2-B) -> Net-(D8-A)
- JP22 pad 3: Net-(JP22-B) -> Net-(JP22-C)
- JP6 pad 1: Net-(JP6-A) -> Net-(D10-K)
- R1 pad 1: 3.3V -> ESP_~{RST}
- R1 pad 2: ESP_~{RST} -> 3.3V
- R10 pad 1: GND -> Net-(J2-CC2)
- R10 pad 2: Net-(J2-CC2) -> GND
- R11 pad 1: Net-(U2-~{RESET}) -> 3.3V_P
- R11 pad 2: 3.3V_P -> Net-(U2-~{RESET})
- R12 pad 1: Net-(JP16-A) -> ESP32/LED_ERROR
- R12 pad 2: ESP32/LED_ERROR -> Net-(JP16-A)
- R13 pad 1: Net-(JP17-A) -> ESP33/LED_LOCK
- R13 pad 2: ESP33/LED_LOCK -> Net-(JP17-A)
- R14 pad 1: GND -> Net-(J4-CC2)
- R14 pad 2: Net-(J4-CC2) -> GND
- R15 pad 1: GND -> Net-(J4-CC1)
- R15 pad 2: Net-(J4-CC1) -> GND
- R16 pad 1: VCCIO -> MCTS2_I
- R16 pad 2: MCTS2_I -> VCCIO
- R17 pad 1: SPEED -> Net-(JP12-B)
- R17 pad 2: Net-(JP12-B) -> SPEED
- R18 pad 1: LINK -> Net-(JP13-B)
- R18 pad 2: Net-(JP13-B) -> LINK
- R19 pad 1: Net-(C11-Pad2) -> TD+
- R19 pad 2: TD+ -> Net-(C11-Pad2)
- R2 pad 1: Net-(Q1B-B2) -> CH340-~{DTR}
- R2 pad 2: CH340-~{DTR} -> Net-(Q1B-B2)
- R20 pad 1: Net-(C11-Pad2) -> TD-
- R20 pad 2: TD- -> Net-(C11-Pad2)
- R21 pad 1: RD- -> Net-(C12-Pad1)
- R21 pad 2: Net-(C12-Pad1) -> RD-
- R22 pad 1: RD+ -> Net-(C12-Pad1)
- R22 pad 2: Net-(C12-Pad1) -> RD+
- R23 pad 1: Net-(U4-COL/CONFIG0) -> 3.3V_P
- R23 pad 2: 3.3V_P -> Net-(U4-COL/CONFIG0)
- R24 pad 1: ETH_~{RST} -> GND
- R24 pad 2: GND -> ETH_~{RST}
- R25 pad 1: Net-(U4-REXT) -> GND
- R25 pad 2: GND -> Net-(U4-REXT)
- R26 pad 1: Net-(U4-REXT) -> GND
- R26 pad 2: GND -> Net-(U4-REXT)
- R27 pad 1: Net-(J6-DAT3/CD) -> 3.3V_P
- R27 pad 2: 3.3V_P -> Net-(J6-DAT3/CD)
- R28 pad 1: SD_CMD -> 3.3V_P
- R28 pad 2: 3.3V_P -> SD_CMD
- R29 pad 1: SD_DATA -> 3.3V_P
- R29 pad 2: 3.3V_P -> SD_DATA
- R3 pad 1: Net-(Q1A-B1) -> CH340-~{RTS}
- R3 pad 2: CH340-~{RTS} -> Net-(Q1A-B1)
- R30 pad 1: 10MHz_1.8V -> Net-(U14-1B)
- R30 pad 2: Net-(U14-1B) -> 10MHz_1.8V
- R31 pad 1: Net-(JP14-B) -> ESP18/SDA2
- R31 pad 2: ESP18/SDA2 -> Net-(JP14-C)
- R32 pad 1: Net-(JP14-A) -> ESP19/SCL2
- R32 pad 2: ESP19/SCL2 -> Net-(JP14-A)
- R33 pad 1: 3.3V_P -> ETH_MDIO
- R33 pad 2: ETH_MDIO -> 3.3V_P
- R34 pad 1: 3.3V_P -> LINK
- R34 pad 2: LINK -> 3.3V_P
- R35 pad 1: 3.3V_P -> SPEED
- R35 pad 2: SPEED -> 3.3V_P
- R36 pad 1: GND -> Net-(JP7-A)
- R36 pad 2: Net-(JP7-A) -> GND
- R37 pad 1: LOG_BTN -> Net-(R37-Pad1)
- R37 pad 2: Net-(R37-Pad2) -> LOG_BTN
- R38 pad 1: Net-(JP18-A) -> 3.3V
- R38 pad 2: 3.3V -> Net-(JP18-A)
- R39 pad 1: Net-(JP19-A) -> LED_RTK
- R39 pad 2: LED_RTK -> Net-(JP19-A)
- R4 pad 1: ESP21/SDA -> Net-(JP1-C)
- R4 pad 2: Net-(JP1-B) -> ESP21/SDA
- R40 pad 1: Net-(JP20-A) -> LED_PVT
- R40 pad 2: LED_PVT -> Net-(JP20-A)
- R41 pad 1: VCCIO -> MRX2_I
- R41 pad 2: MRX2_I -> VCCIO
- R42 pad 1: Net-(JP21-A) -> LED_LOG
- R42 pad 2: LED_LOG -> Net-(JP21-A)
- R43 pad 1: Net-(D15-A2) -> GND
- R43 pad 2: GND -> Net-(D15-A2)
- R44 pad 1: MEventB_I -> GND
- R44 pad 2: GND -> MEventB_I
- R45 pad 1: Net-(E.1-B) -> Net-(E.1-A)
- R45 pad 2: Net-(E.1-A) -> Net-(E.1-B)
- R46 pad 1: Net-(A.1-B) -> Net-(A.1-A)
- R46 pad 2: Net-(A.1-A) -> Net-(A.1-B)
- R47 pad 1: GND -> Net-(V.1-A)
- R47 pad 2: Net-(V.1-A) -> GND
- R48 pad 1: Net-(G.1-B) -> Net-(G.1-A)
- R48 pad 2: Net-(G.1-A) -> Net-(G.1-B)
- R49 pad 1: Net-(C.1-B) -> Net-(C.1-A)
- R49 pad 2: Net-(C.1-A) -> Net-(C.1-B)
- R5 pad 1: Net-(U2-SYNC) -> 1.8V
- R5 pad 2: 1.8V -> Net-(U2-SYNC)
- R50 pad 1: GND -> Net-(C75-Pad2)
- R50 pad 2: Net-(C75-Pad2) -> GND
- R52 pad 1: Net-(R52-Pad1) -> Net-(U17-+)
- R52 pad 2: Net-(U17-+) -> Net-(R52-Pad2)
- R53 pad 1: Net-(U18-EN) -> VCCIO
- R53 pad 2: VCCIO -> Net-(U18-EN)
- R54 pad 1: SDA2_IO -> Net-(JP22-C)
- R54 pad 2: Net-(JP22-B) -> SDA2_IO
- R55 pad 1: SCL2_IO -> Net-(JP22-A)
- R55 pad 2: Net-(JP22-A) -> SCL2_IO
- R56 pad 1: 1.8V -> Net-(D16-A)
- R56 pad 2: Net-(U17--) -> 1.8V
- R57 pad 1: 1.8V -> Net-(U17-+)
- R57 pad 2: Net-(U17-+) -> 1.8V
- R58 pad 1: 10MHz_IN_1.8V -> Net-(R52-Pad2)
- R58 pad 2: Net-(R52-Pad1) -> 10MHz_IN_1.8V
- R59 pad 1: GND -> 10MHz_IN_1.8V
- R59 pad 2: 10MHz_IN_1.8V -> GND
- R6 pad 1: ESP22/SCL -> Net-(JP1-A)
- R6 pad 2: Net-(JP1-A) -> ESP22/SCL
- R7 pad 1: 3.3V -> ESP35/DeviceSense
- R7 pad 2: ESP35/DeviceSense -> 3.3V
- R8 pad 1: ESP35/DeviceSense -> GND
- R8 pad 2: GND -> ESP35/DeviceSense
- R9 pad 1: GND -> Net-(J2-CC1)
- R9 pad 2: Net-(J2-CC1) -> GND
- SW3 pad 2: Net-(R37-Pad2) -> Net-(R37-Pad1)
- U17 pad 1: Net-(R52-Pad1) -> Net-(R52-Pad2)
- U17 pad 4: Net-(U17--) -> Net-(D16-A)
- U6 pad 1: Net-(U6-VIN+) -> Net-(D8-K)
Routing:
- net Net-(JP2-B): track 65.0 -> 0.00 mm, vias 3 -> 0
- net Net-(D8-A): track 0.00 -> 65.0 mm, vias 0 -> 3
- net Net-(U6-VIN+): track 18.1 -> 0.00 mm
- net Net-(D8-K): track 0.00 -> 18.1 mm
- net Net-(JP6-A): track 11.5 -> 0.00 mm
- net Net-(D10-K): track 0.00 -> 11.5 mm
- net Net-(R37-Pad2): track 7.78 -> 0.00 mm
- net Net-(R37-Pad1): track 0.00 -> 7.78 mm
- net Net-(U17--): track 6.32 -> 0.00 mm
- net Net-(D16-A): track 0.00 -> 6.32 mm
- net Net-(JP1-C): track 0.00 -> 6.10 mm, vias 0 -> 1
- net Net-(JP1-B): track 6.10 -> 0.00 mm, vias 1 -> 0
- net Net-(R52-Pad2): track 0.00 -> 3.96 mm
- net Net-(R52-Pad1): track 3.96 -> 0.00 mm
- net GND: track 27.7 -> 30.8 mm
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