File: Hardware/GNSSDO/SparkPNT_GPSDO.kicad_sch (KiCad schematic)
At the start: 49 parts, among them J7 Qwiic_Vertical, J9 Screw_Cage_3.5mm-10, U1 ESP32-WROVER-IE-N16R8

Commit message: KiCad 10
Parts:
- C1: PROD_ID CAP-11015 -> CAP-25001
- C54: PROD_ID CAP-07888 -> CAP-24999
- J7: footprint SparkFun-Connector:JST_SMD_1.0mm-4_Vertical -> SparkFun-Connector:JST_1x04_P1.0mm_Vertical_SMD
- J9: footprint SparkFun-Connector:Screw_Cage_3.5mm-10 -> SparkFun-Connector:ScrewCage_1x10_P3.5mm_Horizontal; symbol SparkFun-Connector:Screw_Cage_3.5mm-10 -> SparkFun-Connector:ScrewCage_1x10_P3.5mm_Green
- JP1, JP15, JP16, JP17, JP18, JP19, JP20, JP21: value ~ -> (none)
- TP1, TP24, TP25, TP26, TP43: footprint SparkFun-Connector:1x01 -> SparkFun-Connector:1x01_P2.54mm
Connections:
- net 3.3V: now also R1.2, R38.1, R7.2; no longer R1.1, R38.2, R7.1
- net ESP21/SDA: now also R4.2; no longer R4.1
- net ESP22/SCL: now also R6.2; no longer R6.1
- net ESP32/LED_ERROR: now also R12.1; no longer R12.2
- net ESP33/LED_LOCK: now also R13.1; no longer R13.2
- net ESP35/DeviceSense: now also R7.1, R8.2; no longer R7.2, R8.1
- net ESP_~{RST}: now also R1.1; no longer R1.2
- net GND: now also R8.1; no longer R8.2
- net LED_LOG: now also R42.1; no longer R42.2
- net LED_PVT: now also R40.1; no longer R40.2
- net LED_RTK: now also R39.1; no longer R39.2
- net at JP18.1 (A): now also R38.2; no longer R38.1
- net at JP1.3 (C): now also R4.1; no longer R4.2
- net at JP20.1 (A): now also R40.2; no longer R40.1
- net at JP1.1 (A): now also R6.1; no longer R6.2
- net at JP19.1 (A): now also R39.2; no longer R39.1
- net at JP16.1 (A): now also R12.2; no longer R12.1
- net at JP17.1 (A): now also R13.2; no longer R13.1
- net at J7.NC1 (NC): no longer J7.NC2 (NC)
- net at JP21.1 (A): now also R42.2; no longer R42.1
- no-connect marks 0 -> 4
Other:
- moved on the sheet: C8, JP1
