File: Hardware/GNSSDO/USB.kicad_sch (KiCad schematic)
At the start: 35 parts, among them J2 USB_C_Receptacle, J4 USB_C_Receptacle, Q1 MBT3904DW1, SW1 PTH_RA_h7.5mm, SW2 PTH_RA_h7.5mm, SW3 PTH_RA_h7.5mm, U3 CH340C

Commit message: KiCad 10
Parts:
- C4: PROD_ID CAP-07888 -> CAP-24999
- D2, D3: symbol SparkFun-DiscreteSemi:D_TVS_ESD_USB -> SparkFun-DiscreteSemi:D_TVS_ESD_USB_5V; Rating (none) -> 5VWM/9VC
- JP10, JP11, JP8, JP9: value ~ -> (none)
- Q1: footprint SparkFun-Semiconductor-Standard:SOT-323 -> SparkFun-Semiconductor-Standard:SOT-363_SC-70-6
- TP34, TP35, TP36, TP37, TP38, TP39, TP46, TP47, TP49, TP50, TP8, TP9: footprint SparkFun-Connector:1x01 -> SparkFun-Connector:1x01_P2.54mm
- TR1: footprint SparkFun-Coil:RFCMF1220100M4T -> SparkFun-Coil:Choke_100MHz_USB
Connections:
- net CH340-~{DTR}: now also R2.1; no longer R2.2
- net CH340-~{RTS}: now also R3.1; no longer R3.2
- net GND: now also R10.2, R14.2, R15.2, R9.2; no longer R10.1, R14.1, R15.1, R9.1
- net LOG_BTN: now also R37.2; no longer R37.1
- net at Q1.2 (B1): now also R3.2; no longer R3.1
- net at J4.A5 (CC1): now also R15.1; no longer R15.2
- net at J4.B5 (CC2): now also R14.1; no longer R14.2
- net at J2.B5 (CC2): now also R10.1; no longer R10.2
- net at SW3.2: now also R37.1; no longer R37.2
- net at Q1.5 (B2): now also R2.2; no longer R2.1
- net at J2.A5 (CC1): now also R9.1; no longer R9.2
- no-connect marks 0 -> 9
Other:
- moved on the sheet: C4, C5, JP8, JP9, TR1
